File: MJ808 clone - all driver.sch (EAGLE design)
At the start: 35 parts, among them IC1 ATTINY4313-MMH, IC2 PRQV8.00CR1510Y00L, IC3 LP38693SD-5.0/NOPB, IC4 LP38693SD-5.0/NOPB, IC5 MCP2515, IC6 MCP2561-2, IC7 MAX16820, Q1 PMV213SN,215, SW1 TL3305-844809

Commit message: - moved PWN line for front light to OC1A, DRC & ERC are ok, updated gerbers
Connections:
- new net N$1: IC1.PCINT17/ICPI-PD6
- new net N$2: IC1.PCINT16/OC0B/T1-PD5
- new net N$3: IC1.AIN1/PCINT1-PB1
- net DIM_FRONT: now also IC1.OC1A/PCINT3-PB3; no longer IC1.PCINT16/OC0B/T1-PD5
- net EN: now also IC1.AIN0/PCINT0-PB0; no longer IC1.OC1A/PCINT3-PB3
Changed lines of the file:
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@@
 </segment>
 <segment>
-<pinref part="IC1" gate="G$1" pin="PCINT16/OC0B/T1-PD5"/>
-<wire x1="170.18" y1="175.26" x2="175.26" y2="175.26" width="0.1524" layer="91"/>
-<label x="175.26" y="175.26" size="1.778" layer="95"/>
+<pinref part="IC1" gate="G$1" pin="OC1A/PCINT3-PB3"/>
+<wire x1="170.18" y1="162.56" x2="175.26" y2="162.56" width="0.1524" layer="91"/>
+<label x="175.26" y="162.56" size="1.778" layer="95"/>
 </segment>
 </net>
@@
 </segment>
 <segment>
-<pinref part="IC1" gate="G$1" pin="OC1A/PCINT3-PB3"/>
-<wire x1="170.18" y1="162.56" x2="175.26" y2="162.56" width="0.1524" layer="91"/>
-<label x="175.26" y="162.56" size="1.778" layer="95"/>
+<pinref part="IC1" gate="G$1" pin="AIN0/PCINT0-PB0"/>
+<wire x1="170.18" y1="170.18" x2="175.26" y2="170.18" width="0.1524" layer="91"/>
+<label x="175.26" y="170.18" size="1.778" layer="95"/>
 </segment>
 </net>
@@
 </segment>
 </net>
+<net name="N$1" class="0">
+<segment>
+<pinref part="IC1" gate="G$1" pin="PCINT17/ICPI-PD6"/>
+<wire x1="170.18" y1="172.72" x2="175.26" y2="172.72" width="0.1524" layer="91"/>
+<label x="175.26" y="172.72" size="1.778" layer="95"/>
+</segment>
+</net>
+<net name="N$3" class="0">
+<segment>
+<pinref part="IC1" gate="G$1" pin="AIN1/PCINT1-PB1"/>
+<wire x1="170.18" y1="167.64" x2="175.26" y2="167.64" width="0.1524" layer="91"/>
+<label x="175.26" y="167.64" size="1.778" layer="95"/>
+</segment>
+</net>
+<net name="N$2" class="0">
+<segment>
+<pinref part="IC1" gate="G$1" pin="PCINT16/OC0B/T1-PD5"/>
+<wire x1="170.18" y1="175.26" x2="175.26" y2="175.26" width="0.1524" layer="91"/>
+<label x="175.26" y="175.26" size="1.778" layer="95"/>
+</segment>
+</net>

Commit message: - rerouted standby pin, updated gerbers
Connections:
- net N$3: now also IC1.OC0A/PCINT2-PB2; no longer IC1.AIN1/PCINT1-PB1
- net STBY: now also IC1.AIN1/PCINT1-PB1; no longer IC1.OC0A/PCINT2-PB2
Changed lines of the file:
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@@
 </segment>
 <segment>
-<pinref part="IC1" gate="G$1" pin="OC0A/PCINT2-PB2"/>
-<wire x1="170.18" y1="165.1" x2="175.26" y2="165.1" width="0.1524" layer="91"/>
-<label x="175.26" y="165.1" size="1.778" layer="95"/>
+<pinref part="IC1" gate="G$1" pin="AIN1/PCINT1-PB1"/>
+<wire x1="170.18" y1="167.64" x2="175.26" y2="167.64" width="0.1524" layer="91"/>
+<label x="175.26" y="167.64" size="1.778" layer="95"/>
 </segment>
 </net>
@@
 </segment>
 </net>
-<net name="N$3" class="0">
-<segment>
-<pinref part="IC1" gate="G$1" pin="AIN1/PCINT1-PB1"/>
-<wire x1="170.18" y1="167.64" x2="175.26" y2="167.64" width="0.1524" layer="91"/>
-<label x="175.26" y="167.64" size="1.778" layer="95"/>
-</segment>
-</net>
 <net name="N$2" class="0">
 <segment>
@@
 </segment>
 </net>
+<net name="N$3" class="0">
+<segment>
+<pinref part="IC1" gate="G$1" pin="OC0A/PCINT2-PB2"/>
+<wire x1="170.18" y1="165.1" x2="175.26" y2="165.1" width="0.1524" layer="91"/>
+<label x="175.26" y="165.1" size="1.778" layer="95"/>
+</segment>
+</net>

Commit message: - fine-tuned POC and final board, they are in sync, ERC & DRC check out, updated gerbers, cleaned up BOM
Parts:
- removed IC7: MAX16820, MAX16820 LED Driver, constant current:MAX16820
- removed R12: 120, rcl:R-EU_R0805
- added C3: 100μF, rcl:C-EUC1206
- added C6: 47μF, rcl:C-EUC0805
- C1: value 0.1μF -> 1μF
- C2, C5: value 22μF -> 1μF; device rcl:C-EUC0603 -> rcl:C-EUC0402
- C4: value 47μF / 15V+ -> 47μF
- IC2: value PRQV8.00CR1510Y00L -> PRQV8.00CR1510Y00L
- IC3: value LP38693SD-5.0/NOPB -> MCP2515; device LP38693 5V LDO:LP38693 -> MCP2515-I-ML - Standalonce CAN Controller with SPI Interface:MCP2515-I-ML
- IC5: value MCP2515 -> MCP2561-2; device MCP2515-I-ML - Standalonce CAN Controller with SPI Interface:MCP2515-I-ML -> MCP2561-2 - High-Speed CAN Transceiver:MCP2561-2
- IC6: value MCP2561-2 -> MAX16820; device MCP2561-2 - High-Speed CAN Transceiver:MCP2561-2 -> MAX16820 LED Driver, constant current:MAX16820
- R10: value 0.15 / 1W -> 10k; device rcl:R-EU_R1210 -> rcl:R-EU_R0402
- R11: value 10k -> 120; device rcl:R-EU_R0402 -> rcl:R-EU_R0805
- R3, R6: value 10k -> 330
- R4, R7: value 330 -> 10k
- R9: value 10k -> 0.15 / 1W; device rcl:R-EU_R0402 -> rcl:R-EU_R1210
Connections:
- removed net 5V0_CAN: C2.1, IC3.OUT, IC3.SNS, IC5.VDD, IC6.VCC, R11.1, R6.1
- removed net 5V0_μC: C1.1, C5.2, IC1.VCC, IC4.OUT, ICSP.5, R2.2, SW1.P$1
- removed net EN: IC1.AIN0/PCINT0-PB0, IC3.EN, R3.2
- new net 5V0: C1.1, C2.1, C3.2, C5.1, IC1.VCC, IC3.VDD, IC4.OUT, IC5.VCC, ICSP.5, R10.1, R2.2, R4.1, SW1.P$1
- new net N$4: IC1.AIN0/PCINT0-PB0
- net BAT+: now also C4.2, C6.1, IC6.IN, R9.2; no longer C4.1, IC3.IN, IC7.IN, R10.2
- net CANH: now also IC5.CANH, R11.2; no longer IC6.CANH, R12.2
- net CANL: now also IC5.CANL, R11.1; no longer IC6.CANL, R12.1
- net CLOCKOUT: now also IC3.OSC1; no longer IC5.OSC1
- net DIM_FRONT: now also IC6.DIM, R8.1; no longer IC7.DIM, R9.1
- net DIM_FRONT_GATE: now also IC6.DRV, R7.1; no longer IC7.DRV, R8.1
- net GATE: now also R7.2; no longer R8.2
- net GND: now also C3.1, C4.1, C5.2, C6.2, R8.2; no longer C4.2, C5.1, IC7.GND, R3.1, R9.2
- net ICSP_MISO: now also R6.2; no longer R7.2
- net ICSP_SCK: now also R3.2; no longer R4.2
- net INT: now also IC3.!INT!; no longer IC5.!INT!
- net LED_AN: now also IC6.CS, R9.1; no longer IC7.CS, R10.1
- net RXCAN: now also IC3.RXCAN, IC5.RXD; no longer IC5.RXCAN, IC6.RXD
- net SPI_MISO: now also IC3.SO, R6.1; no longer IC5.SO, R7.1
- net SPI_MOSI: now also IC3.SI; no longer IC5.SI
- net SPI_SCK: now also IC3.SCK, R3.1; no longer IC5.SCK, R4.1
- net SPI_SS: now also IC3.!CS!, R4.2; no longer IC5.!CS!, R6.2
- net STBY: now also IC5.STBY, R10.2; no longer IC6.STBY, R11.2
- net TXCAN: now also IC3.TXCAN, IC5.TXD; no longer IC5.TXCAN, IC6.TXD
Other:
- note removed: "power supply for CAN infrastructure"
- moved on the sheet: C2, C4, C5, R10, R11, R3, R4, R6, R7, R8, R9
