File: cos POC.brd (EAGLE design)
At the start: 100 x 35.5 mm, 66 parts, among them IC1 LM74670QDGKRQ1, IC11 LM74670QDGKRQ1, IC2 LM74670QDGKRQ1, IC3 LM74670QDGKRQ1, IC4 SQJ960EP N-FET, IC5 SQJ960EP N-FET, IC6 ATTINY4313-MMH, IC7 PRQV8.00CR1510Y00L, IC8 MCP2515, IC9 MCP2561-2

Commit message: - further work on cos schematic
Parts:
- removed R2: 741X083331JP 330R, 74x-1133528 Resistor Array:0402
- added C21: 1μF, rcl:C0402
- added IC10: (no value), TS5A1066 Analogue Switch IC:SOT-23
- added R19: 741X083331JP 330R, 74x-1133528 Resistor Array:0402
- IC12: value (none) -> LTC3350
- moved R1 84.8 mm to (74.5, 30.2), flipped to the bottom, turned to 180 degrees
- moved C7 84.5 mm to (70.5, 24.5), flipped to the bottom
- moved C8 74.1 mm to (74.2, 22.0), flipped to the bottom
- moved IC9 61.7 mm to (74.2, 26.0), flipped to the bottom
- moved IC7 48.4 mm to (88.5, 12.5), flipped to the bottom
- moved C9 42.5 mm to (83.8, 15.8), flipped to the bottom, turned to 270 degrees
- moved CAN 38.8 mm to (74.5, 33.0), turned to 180 degrees
- renumbered BAT to 6V0
Connections:
- net BAT+ renamed 6V0
- net N$7 renamed !PFO!
- removed net 5V0_REG: C7.1, C8.1, IC8.VDD, IC9.VDD
- removed net DIM_BRAKE: R3.6
- removed net N$1: IC12.SCL
- removed net N$2: IC12.SDA
- removed net N$6: IC12.!SMBALERT!
- removed net N$8: IC12.CAPFB
- new net !SMBALERT!: IC12.!SMBALERT!, IC6.12
- new net CAPGD: IC12.CAPGD
- new net I2C_SDA: IC10.2, IC12.SDA
- new net VCC2P5: C21.1, IC12.CAP_SLCT1, IC12.CAP_SLCTO, IC12.VCC2P5
- net 5V0: now also C7.1, C8.1, IC10.5, IC8.VDD, IC9.VDD, R19.7; no longer R3.7
- net GND: now also C21.2, IC10.3; no longer IC12.CAP_SLCTO, R3.5
- net ICSP_DI/MISO: now also IC10.1, R19.6; no longer R2.5
- net ICSP_DO/MOSI: now also R19.4; no longer R2.3
- net ICSP_SCK: now also IC12.SCL, R19.2; no longer R2.1
- net N$38: now also IC12.CAPFB; no longer IC12.CAPDG
- net SPI_MISO: now also R19.5; no longer R2.6
- net SPI_MOSI: now also R19.3; no longer R2.4
- net SPI_SCK: now also R19.1; no longer R2.2
- net SPI_SS: now also IC10.4, R19.8; no longer R3.8
Routing:
- net CKOUT: track 2.78 -> 22.3 mm, vias 1 -> 0
- net SPI_SS: track 0.00 -> 16.1 mm
- net 5V0: track 3.70 -> 14.6 mm, vias 1 -> 3
- net ICSP_DI/MISO: track 5.42 -> 14.3 mm, vias 1 -> 2
- net TXCAN: track 0.00 -> 3.77 mm, vias 0 -> 1
- net RXCAN: track 0.00 -> 3.75 mm, vias 0 -> 1
- net XTAL1: track 2.56 -> 4.74 mm
- net XTAL2: track 2.58 -> 4.76 mm
- net ICSP_DO/MOSI: track 4.52 -> 6.52 mm, vias 1 -> 0
- net ICSP_SCK: track 4.93 -> 6.62 mm, vias 1 -> 0
- net SPI_MOSI: track 1.85 -> 2.89 mm, vias 1 -> 0
- net SPI_MISO: track 2.50 -> 2.85 mm, vias 1 -> 0
- net SPI_SCK: track 2.96 -> 2.85 mm, vias 1 -> 0

Commit message: - replaced LTC3350 with LTC3351, updated schematic and board
Parts:
- removed 6V0: BAT, con-molex:22-23-2021
- removed C10, C11, C12, C16, C17, C18, C19: 0.1μF, rcl:C0402
- removed C15: 10μF, rcl:C0402
- removed C20: 4.7n, rcl:C0402
- removed C21: 1μF, rcl:C0402
- removed CAN: CAN, con-molex:22-23-2021
- removed DYNAMO: 22-27-2021-02, con-molex:6410-02
- removed IC1: LM74670QDGKRQ1, LM74670 - Smart Diode Rectifier Controller:VSSOP-8
- removed IC4, IC5: SQJ960EP N-FET, SQJ96XEP - MosFET:SO-8L
- removed JP12: (no value), pinhead:1X01
- removed R12, R15, R16: 2.7, rcl:R0402
- removed R17, R18, R5: 121, rcl:R0402
- removed R19: 741X083331JP 330R, 74x-1133528 Resistor Array:0402
- removed R6: 88.7k, rcl:R0402
- removed R7: 2k, rcl:R0402
- removed U$1, U$2: SIA456DJ, SIA456DJ-T1-GE3 N-Fet:SC-70-6
- added C27, C33: 0.1μF, rcl:C0805
- added C32, C_F: 0.1μF, rcl:C0402
- added CAP1, CAP2, CAP3, CAP4: 15F, rcl:E5-8,5
- added C_C: 4.7nF, rcl:C0402
- added C_CAP1, C_CAP2, C_CAP3, C_CAP4, C_SS: 22μF, rcl:C0402
- added C_CP5: 1μF, rcl:C0402
- added C_OUT1-1, C_OUT1-2, C_OUT1-3, C_OUT1-4, C_OUT1-5, C_OUT1-6: 100μF, rcl:C0402
- added C_OUT2-1, C_OUT2-2: 2.2μF, rcl:C0402
- added D3: CZRB5349B-HF, zener:DO-214
- added IC13: LM74670QDGKRQ1, LM74670 - Smart Diode Rectifier Controller:VSSOP-8
- added IC14: MCP2561-2, MCP2561-2 - High-Speed CAN Transceiver:DFN10
- added IC15: (no value), TS5A1066 Analogue Switch IC:SOT-23
- added IC16, MN1, MN2, MN3, MN5: (no value), SIA456DJ-T1-GE3 N-Fet:SC-70-6
- added J1: 22-27-2021-02, con-molex:6410-02
- added JP6: (no value), pinhead:1X02
- added L1: 10μH, rcl:L1812
- added R2: 2k, rcl:R0402
- added R23: 741X083102JP 10k, 74x-1133528 Resistor Array:0402-4R
- added R24: 741X083331JP 330R, 74x-1133528 Resistor Array:0402-4R
- added R25: 330k, rcl:R0805
- added R26: 120, rcl:R0805
- added R_CAP1, R_CAP2, R_CAP3, R_CAP4, R_CAPRTN: 2.7Ω, rcl:R0402
- added R_FB01: 400k, rcl:R0402
- added R_FB02: 100k, rcl:R0402
- added R_FBC1: 732k, rcl:R0402
- added R_FBC2: 274k, rcl:R0402
- added R_PF1, R_PF3: 30.1k, rcl:R0402
- added R_PF2: 10k, rcl:R0402
- added R_SNSC: 0.003Ω, rcl:R0402
- added R_SNSI: 0.064Ω, rcl:R0402
- added R_T: 88.7k, rcl:R0402
- added R_T1: 100k THERM, rcl:R0402
- added R_TST: 20Ω, rcl:R0402
- added X1: CAN, con-molex:22-23-2021
- added X2: BAT, con-molex:22-23-2021
- C1: value 0.1μF -> 1μF; device rcl:C0805 -> rcl:C0402
- C13: value 0.1μF -> 4.7μF
- C3: value 0.1μF -> 4.7nF; device rcl:C0805 -> rcl:C0402
- C5: value (none) -> 100pF
- C6: value 4.7n -> 0.1μF
- D1: value CZRB5349B-HF -> (none); device zener:DO-214 -> diode:SMC
- IC10: value (none) -> MCP2515; device TS5A1066 Analogue Switch IC:SOT-23 -> MCP2515-I-ML - Standalonce CAN Controller with SPI Interface:QFN20
- IC11: value LM74670QDGKRQ1 -> PRQV8.00CR1510Y00L; device LM74670 - Smart Diode Rectifier Controller:VSSOP-8 -> PRQV8.00CR1510Y00L - 8MHz resonator:SMT
- IC12: value LTC3350 -> SQJ960EP N-FET; device LTC3350fc High Current Supercapacitor Backup Controller and System Monitor:QFN38 -> SQJ96XEP - MosFET:SO-8L
- IC3: value LM74670QDGKRQ1 -> (none); device LM74670 - Smart Diode Rectifier Controller:VSSOP-8 -> LTC3351f - Hot Swappable Supercapacitor Charger, Backup Controller and System Monitor:QFN44
- IC6: value ATTINY4313-MMH -> LM74670QDGKRQ1; device ATtiny4313 microcontroller:VQFN-20 -> LM74670 - Smart Diode Rectifier Controller:VSSOP-8
- IC7: value PRQV8.00CR1510Y00L -> ATTINY4313-MMH; device PRQV8.00CR1510Y00L - 8MHz resonator:SMT -> ATtiny4313 microcontroller:VQFN-20
- IC8: value MCP2515 -> LM74670QDGKRQ1; device MCP2515-I-ML - Standalonce CAN Controller with SPI Interface:QFN20 -> LM74670 - Smart Diode Rectifier Controller:VSSOP-8
- IC9: value MCP2561-2 -> SQJ960EP N-FET; device MCP2561-2 - High-Speed CAN Transceiver:DFN10 -> SQJ96XEP - MosFET:SO-8L
- JP1: value (none) -> JUMPER-SMT_2_NO_SILK; device pinhead:1X02 -> SparkFun-Jumpers:SMT-JUMPER_2_NO_SILK
- JP3: value JUMPER-SMT_2_NO_SILK -> (none); device SparkFun-Jumpers:SMT-JUMPER_2_NO_SILK -> pinhead:1X02
- JP8: device pinhead:1X02 -> pinhead:1X01
- R1: value 120 -> 100k; device rcl:R0805 -> rcl:R0402
- R10, R11: value 2.7 -> 10Ω
- R13, R14: value 2.7 -> 10k
- R3: value 741X083102JP 10k -> 10k; device 74x-1133528 Resistor Array:0402 -> rcl:R0402
- R4: value (none) -> 10k
- R8: value 2k -> 10k
- R9: value 330k -> 100Ω; device rcl:R0805 -> rcl:R0402
- moved R14 219.4 mm to (55.2, 21.0), flipped to the bottom, turned to 270 degrees
- moved R13 218.2 mm to (55.2, 23.2), flipped to the bottom, turned to 90 degrees
- moved R11 212.2 mm to (47.2, 26.0), flipped to the bottom, turned to 180 degrees
- moved R10 210.0 mm to (47.2, 27.2), flipped to the bottom
- moved C13 177.0 mm to (58.0, 20.0), flipped to the bottom, turned to 90 degrees
- moved R8 156.5 mm to (35.5, 23.5), flipped to the bottom, turned to 180 degrees
- moved C6 151.6 mm to (55.2, 17.5), flipped to the bottom, turned to 270 degrees
- moved R4 134.2 mm to (35.5, 20.5), flipped to the bottom, turned to 180 degrees
- moved C5 130.3 mm to (32.2, 17.2), flipped to the bottom, turned to 180 degrees
- moved JP4 96.4 mm to (22.0, 19.0), turned to 0 degrees
- moved R3 95.0 mm to (35.5, 22.0), flipped to the bottom, turned to 180 degrees
- moved JP8 92.5 mm to (23.2, 28.5)
- moved JP3 85.7 mm to (90.2, -35.2)
- moved IC6 80.1 mm to (9.75, 4.75), turned to 180 degrees
- moved JP5 77.7 mm to (26.5, -5.75), turned to 0 degrees
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- renumbered C14 to C31, C2 to C30, C4 to C34, C8 to C29, C9 to C28, IC2 to IC17, JP11 to JP7, SPI to CONN1, SPLIT to TP1
Connections:
- removed net N$17: C6.2, R7.2
- removed net N$21: IC12.GPI
- removed net N$22: C10.1, IC12.CFP
- removed net N$23: C10.2, IC12.CFN
- removed net N$24: C11.1, IC12.VCAP
- removed net N$25: C11.2, IC12.VCAPP5
- removed net N$26: C12.2, IC12.TGATE
- removed net N$28: C13.1, C15.1, IC12.DRVCC, IC12.INTVCC
- removed net N$29: C16.1, C17.2, R10.2
- removed net N$30: C17.1, C18.2, R11.2
- removed net N$31: C18.1, C19.2, R12.2
- removed net N$32: IC12.CAP1, R10.1
- removed net N$33: IC12.CAP2, R11.1
- removed net N$34: IC12.CAP3, R12.1
- removed net N$35: IC12.CAP4, R13.1
- removed net N$36: C19.1, R13.2, R15.1
- removed net N$37: IC12.CAPRTN, R14.1
- removed net N$38: IC12.CAPFB, R15.2, R16.1
- removed net N$39: IC12.PFI, R17.2, R18.1
- removed net N$40: C20.2, IC12.VIN
- removed net N$41: R17.1
- removed net N$5: JP1.2, JP3.2
- new net BGATE: IC3.30-BGATE, MN3.3G
- new net BST: C6.1, D1.C, IC3.29-BST
- new net CAP1: IC3.16-CAP1, R_CAP1.1
- new net CAP2: IC3.17-CAP2, R_CAP2.1
- new net CAP3: IC3.18-CAP3, R_CAP3.1
- new net CAP4: IC3.19-CAP4, R_CAP4.1
- new net CAPFB: IC3.9-CAPFB, R_FBC1.1, R_FBC2.2
- new net CAPRTN: IC3.15-CAPRTN, R_CAPRTN.1
- new net CFN: C_F.2, IC3.21-CFN
- new net CFP: C_F.1, IC3.20-CFP
- new net CSS: C_SS.2, IC3.38_CSS
- new net CTIMER: C3.2, IC3.44-CTIMER
- new net DRVCC: C13.1, C7.1, D1.A, IC3.31-DRVCC, IC3.32-INTVCC
- new net GPI: IC3.13-GPI, R1.2, R_T1.1
- new net ICAP: IC3.25-ICAP, L1.2, R_SNSC.1
- new net ITST: IC3.14-ITST, R_TST.1
- new net N$1: IC3.39_SRC, MN1.4S, MN1.S, MN5.4S, MN5.S
- new net N$2: MN1.3G, R10.1
- new net N$6: IC3.36-ISNSP_CHG, IC3.37-ISNS_HS, MN5.1D, MN5.2D, MN5.5D, MN5.6D, MN5.D, R_SNSI.1
- new net N$7: CAP3.+, CAP4.-, R_CAP3.2
- new net N$8: CAP2.+, CAP3.-, R_CAP2.2
- new net OUTFB: C5.2, IC3.10-OUTFB, R_FB01.2, R_FB02.1
- new net OV: IC3.43-OV, R_PF2.2, R_PF3.1
- new net RETRYB: IC3.34-RETRYB, R13.1, R14.1
- new net RT: IC3.12-RT, R_T.1
- new net SW: C6.2, IC3.27-SW, L1.1, MN2.4S, MN2.S, MN3.1D, MN3.2D, MN3.5D, MN3.6D, MN3.D
- new net TGATE: IC3.28-TGATE, MN2.3G
- new net UV: IC3.42-UV, R_PF1.2, R_PF2.1
- new net VC: IC3.8-VC, R2.1
- new net VCAP: CAP4.+, C_CAP1.1, C_CAP2.1, C_CAP3.1, C_CAP4.1, C_CP5.1, IC3.24-VCAP, R_CAP4.2, R_FBC1.2, R_SNSC.2
- new net VCAPP5: C_CP5.2, IC3.22-VCAPP5
- new net VDD: R3.1, R4.1, R8.1
- new net VIN: MN1.1D, MN1.2D, MN1.5D, MN1.6D, MN1.D, R9.2, R_PF1.1
- new net VOUT: C5.1, C_OUT1-1.1, C_OUT1-2.1, C_OUT1-3.1, C_OUT1-4.1, C_OUT1-5.1, C_OUT1-6.1, C_OUT2-1.1, C_OUT2-2.1, C_SS.1, IC3.33-VOUT, IC3.35-ISNSM, MN2.1D, MN2.2D, MN2.5D, MN2.6D, MN2.D, R14.2, R_FB01.1, R_SNSI.2
- net !PFO!: now also IC3.3-VINGD, R8.2; no longer IC12.!PFO!
- net !SMBALERT!: now also IC3.6-!SMBALERT!, IC7.12, R3.2; no longer IC12.!SMBALERT!, IC6.12
- net 5V0: now also C32.1, IC10.VDD, IC14.VDD, IC15.5, IC7.18, R23.1, R23.3, R24.7, R25.2; no longer C7.1, IC10.5, IC6.18, IC8.VDD, IC9.VDD, R19.7, R3.1, R3.3, R9.2
- net 6V0: now also X2.2; no longer 6V0.2
- net CANH: now also IC14.CANH, R26.2, X1.1; no longer CAN.1, IC9.CANH, R1.2
- net CANL: now also IC14.CANL, R26.1, X1.2; no longer CAN.2, IC9.CANL, R1.1
- net CAPGD: now also IC3.7-CAPGD, R4.2; no longer IC12.CAPGD
- net CKOUT: now also IC10.OSC1, IC7.4; no longer IC6.4, IC8.OSC1
- net DEBUGWIRE/RESET: now also IC7.19; no longer IC6.19
- net DYNAMO_1: now also D3.AN, IC6.CATHODE, IC8.ANODE, IC9.D1, IC9.S2, J1.1; no longer D2.AN, DYNAMO.1, IC1.CATHODE, IC3.ANODE, IC5.D1, IC5.S2
- net DYNAMO_2: now also D2.AN, IC12.D2, IC12.S1, IC13.ANODE, IC16.3G, J1.2; no longer D1.AN, DYNAMO.2, IC11.ANODE, IC4.D2, IC4.S1, U$1.G
- net FET1_G: now also IC6.GATE_DRIVE, IC6.GATE_PULLD, IC9.G1; no longer IC1.GATE_DRIVE, IC1.GATE_PULLD, IC5.G1
- net FET2_G: now also IC8.GATE_DRIVE, IC8.GATE_PULLD, IC9.G2; no longer IC3.GATE_DRIVE, IC3.GATE_PULLD, IC5.G2
- net FET3_G: now also IC12.G1, IC13.GATE_DRIVE, IC13.GATE_PULLD; no longer IC11.GATE_DRIVE, IC11.GATE_PULLD, IC4.G1
- net FET4_G: now also IC12.G2; no longer IC4.G2
- net GND: now also C1.2, C3.1, C32.2, CAP1.-, C_C.2, C_CAP1.2, C_CAP2.2, C_CAP3.2, C_CAP4.2, C_OUT1-1.2, C_OUT1-2.2, C_OUT1-3.2, C_OUT1-4.2, C_OUT1-5.2, C_OUT1-6.2, C_OUT2-1.2, C_OUT2-2.2, IC10.GND, IC10.GND6, IC11.GND, IC12.S2, IC14.GND, IC14.VSS, IC15.3, IC16.4S, IC16.S, IC3.11SGND, IC3.GND10, IC3.GND2, IC3.GND3, IC3.GND4, IC3.GND5, IC3.GND6, IC3.GND7, IC3.GND8, IC3.GND9, IC3.PGND, IC6.ANODE, IC7.8, IC9.S1, JP6.2, MN3.4S, MN3.S, R13.2, R_CAPRTN.2, R_FB02.2, R_FBC2.1, R_PF3.2, R_T.2, R_T1.2, R_TST.2, X2.1; no longer 6V0.1, C15.2, C16.2, C20.1, C21.2, IC1.ANODE, IC10.3, IC12.GND0, IC12.GND1, IC12.GND2, IC12.GND3, IC12.GND4, IC12.GND5, IC12.GND6, IC12.GND7, IC12.GND8, IC12.GND9, IC12.SGND, IC4.S2, IC5.S1, IC6.8, IC6.GND, IC8.GND, IC8.GND6, IC9.GND, IC9.VSS, JP3.1, R14.2, R18.2, R5.2, U$1.S
- net I2C_SDA: now also IC15.2, IC3.5-SDA; no longer IC10.2, IC12.SDA
- net ICSP_DI/MISO: now also IC15.1, IC7.15, R24.6; no longer IC10.1, IC6.15, R19.6
- net ICSP_DO/MOSI: now also IC7.16, R24.4; no longer IC6.16, R19.4
- net ICSP_SCK: now also IC3.4-SCL, IC7.17, R24.2; no longer IC12.SCL, IC6.17, R19.2
- net INT1: now also IC10.!INT!, IC7.5; no longer IC6.5, IC8.!INT!
- net N$12: now also C33.1, IC13.VCAPL; no longer C3.1, IC11.VCAPL
- net N$13: now also C33.2, IC13.VCAPH; no longer C3.2, IC11.VCAPH
- net N$14: now also IC8.VCAPL; no longer IC3.VCAPL
- net N$15: now also IC8.VCAPH; no longer IC3.VCAPH
- net N$16: now also CAP1.+, CAP2.-, R_CAP1.2; no longer IC12.ITST, R5.1
- net N$18: now also MN5.3G, R11.2; no longer IC12.RT, R6.1
- net N$19: now also C_C.1, R2.2; no longer C6.1, R6.2
- net N$20: now also IC3.40-HS_GATE, R10.2, R11.1; no longer IC12.VC, R7.1
- net N$27: now also IC3.41-VIN, R9.1; no longer C12.1, IC12.BST
- net N$3: now also C27.2, IC6.VCAPH; no longer C1.2, IC1.VCAPH
- net N$4: now also JP4.2, JP6.1; no longer JP1.1, JP2.2
- net N$9: now also C27.1, IC6.VCAPL; no longer C1.1, IC1.VCAPL
- net OUT+: now also IC12.D1, IC13.CATHODE, IC8.CATHODE, IC9.D2, JP4.1; no longer IC11.CATHODE, IC3.CATHODE, IC4.D1, IC5.D2, JP2.1
- net RESET: now also IC10.!RESET!, R23.4; no longer IC8.!RESET!, R3.4
- net RXCAN: now also IC10.RXCAN, IC14.RXD; no longer IC8.RXCAN, IC9.RXD
- net SPI_MISO: now also IC10.SO, R24.5; no longer IC8.SO, R19.5
- net SPI_MOSI: now also IC10.SI, R24.3; no longer IC8.SI, R19.3
- net SPI_SCK: now also IC10.SCK, R24.1; no longer IC8.SCK, R19.1
- net SPI_SS: now also IC10.!CS!, IC15.4, IC7.14, R24.8; no longer IC10.4, IC6.14, IC8.!CS!, R19.8
- net SPLIT: now also IC14.SPLIT; no longer IC9.SPLIT
- net STBY: now also IC14.STBY, IC7.11, R23.2; no longer IC6.11, IC9.STBY, R3.2
- net TXCAN: now also IC10.TXCAN, IC14.TXD; no longer IC8.TXCAN, IC9.TXD
- net VCC2P5: now also C1.1, IC3.1-CAP_SLCT0, IC3.2-CAP_SLCT1, IC3.26-VCC2P5, R1.1; no longer C21.1, IC12.CAP_SLCT1, IC12.CAP_SLCTO, IC12.VCC2P5
- net XTAL1: now also IC11.XTAL1, IC7.3; no longer IC6.3, IC7.XTAL1
- net XTAL2: now also IC11.XTAL2, IC7.2; no longer IC6.2, IC7.XTAL2
- net ZENER_COMMON: now also D3.CAT; no longer D1.CAT
- net ZERO_CROSS: now also IC16.1D, IC16.2D, IC16.5D, IC16.6D, IC16.D, JP8.1, R25.1; no longer JP12.1, R9.1, U$1.D
Routing:
- net VCC2P5: track 0.00 -> 39.4 mm, vias 0 -> 3
- net CAP4: track 0.00 -> 23.4 mm, vias 0 -> 1
- net CAPRTN: track 0.00 -> 18.4 mm, vias 0 -> 1
- net DRVCC: track 0.00 -> 17.8 mm, vias 0 -> 1
- net BST: track 0.00 -> 15.3 mm, vias 0 -> 1
- net OUTFB: track 0.00 -> 15.2 mm, vias 0 -> 1
- net CAP3: track 0.00 -> 14.2 mm, vias 0 -> 1
- net CAP1: track 0.00 -> 14.0 mm, vias 0 -> 1
- net VCAP: track 0.00 -> 13.6 mm, vias 0 -> 1
- net VOUT: track 0.00 -> 11.0 mm, vias 0 -> 2
- net GPI: track 0.00 -> 10.4 mm, vias 0 -> 1
- net ITST: track 0.00 -> 9.96 mm, vias 0 -> 1
- net DYNAMO_2: track 35.8 -> 25.9 mm
- net DYNAMO_1: track 23.6 -> 13.8 mm
- net RETRYB: track 0.00 -> 9.22 mm, vias 0 -> 1
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- added copper zone on layer 1, net DYNAMO_1
- added copper zone on layer 1, net DYNAMO_2
- added copper zone on layer 1, net GND
- added copper zone on layer 16, net GND
- added copper zone on layer 1, net VOUT

Commit message: - continued work on POC board
Parts:
- removed JP2, JP5: JUMPER-SMT_2_NO_SILK, SparkFun-Jumpers:SMT-JUMPER_2_NO_SILK
- removed JP3: (no value), pinhead:1X02
- removed TP1: TPB2,54, testpad:B2,54
- moved MN3 74.0 mm to (57.8, 43.8), turned to 270 degrees
- moved C_OUT2-2 72.3 mm to (55.8, 44.5), turned to 270 degrees
- moved C_OUT2-1 70.9 mm to (54.5, 44.5), turned to 270 degrees
- moved C_OUT1-6 68.9 mm to (52.8, 44.5), turned to 270 degrees
- moved C_OUT1-5 67.5 mm to (51.5, 44.5), turned to 270 degrees
- moved C_OUT1-4 66.1 mm to (50.2, 44.5), turned to 270 degrees
- moved C_OUT1-3 64.7 mm to (49.0, 44.5), turned to 270 degrees
- moved C_OUT1-2 63.4 mm to (47.8, 44.5), turned to 270 degrees
- moved C_OUT1-1 62.1 mm to (46.5, 44.5), turned to 270 degrees
- moved MN2 61.3 mm to (44.5, 45.8), turned to 180 degrees
- moved R_SNSI 58.8 mm to (42.2, 45.5), turned to 0 degrees
- moved L1 42.1 mm to (57.0, 14.0), flipped to the bottom, turned to 180 degrees
- moved R_SNSC 38.5 mm to (62.0, 14.0), flipped to the bottom, turned to 180 degrees
- moved X1 15.2 mm to (74.2, 30.0)
- moved X2 13.6 mm to (68.0, 30.0), turned to 180 degrees
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Connections:
- removed net SPLIT: IC14.SPLIT, TP1.TP
- removed net VOUT: C5.1, C_OUT1-1.1, C_OUT1-2.1, C_OUT1-3.1, C_OUT1-4.1, C_OUT1-5.1, C_OUT1-6.1, C_OUT2-1.1, C_OUT2-2.1, C_SS.1, IC3.33-VOUT, IC3.35-ISNSM, MN2.1D, MN2.2D, MN2.5D, MN2.6D, MN2.D, R14.2, R_FB01.1, R_SNSI.2
- net 6V0: now also C5.1, C_OUT1-1.1, C_OUT1-2.1, C_OUT1-3.1, C_OUT1-4.1, C_OUT1-5.1, C_OUT1-6.1, C_OUT2-1.1, C_OUT2-2.1, C_SS.1, IC3.33-VOUT, IC3.35-ISNSM, MN2.1D, MN2.2D, MN2.5D, MN2.6D, MN2.D, R14.2, R_FB01.1, R_SNSI.2
- net N$4: now also JP1.1
- net VIN: now also JP1.2
Routing:
- net VOUT: track 11.0 -> 0.00 mm, vias 2 -> 0
- net 6V0: track 0.00 -> 11.0 mm, vias 0 -> 2
- net CANL: track 0.00 -> 5.47 mm
- net CANH: track 0.00 -> 5.47 mm
- net N$4: track 3.10 -> 6.20 mm
- net GND: vias 7 -> 11
- added copper zone on layer 1, net 6V0
- removed copper zone on layer 1, net VOUT
Other:
- outline, holes or cut-outs redrawn
