File: cos POC.sch (EAGLE design)
At the start: 66 parts, among them IC1 LM74670QDGKRQ1, IC11 LM74670QDGKRQ1, IC2 LM74670QDGKRQ1, IC3 LM74670QDGKRQ1, IC4 SQJ960EP N-FET, IC5 SQJ960EP N-FET, IC6 ATTINY4313-MMH, IC7 PRQV8.00CR1510Y00L, IC8 MCP2515, IC9 MCP2561-2

Commit message: - further work on cos schematic
Parts:
- removed R2: 741X083331JP 330R, 74x-1133528 Resistor Array:741X083331JP
- added C21: 1μF, rcl:C-EUC0402
- added IC10: (no value), TS5A1066 Analogue Switch IC:TS5A1066SOT-23
- added R19: 741X083331JP 330R, 74x-1133528 Resistor Array:741X083331JP
- IC12: value (none) -> LTC3350
- renumbered BAT to 6V0
Connections:
- net BAT+ renamed 6V0
- net N$7 renamed !PFO!
- net N$8 renamed CAPGD
- removed net 5V0_REG: C7.1, C8.1, IC8.VDD, IC9.VCC
- removed net DIM_BRAKE: R3.6
- removed net N$1: IC12.SCL
- removed net N$2: IC12.SDA
- removed net N$6: IC12.!SMBALERT!
- new net !SMBALERT!: IC12.!SMBALERT!, IC6.OC0A/PCINT2-PB2
- new net I2C_SDA: IC10.COM, IC12.SDA
- new net VCC2P5: C21.1, IC12.CAP_SLCT0, IC12.CAP_SLCT1, IC12.VCC2P5
- net 5V0: now also C7.1, C8.1, IC10.VCC, IC8.VDD, IC9.VCC, R19.7; no longer R3.7
- net GND: now also C21.2, IC10.GND; no longer IC12.CAP_SLCT1, R3.5
- net ICSP_DI/MISO: now also IC10.NO, R19.6; no longer R2.5
- net ICSP_DO/MOSI: now also R19.4; no longer R2.3
- net ICSP_SCK: now also IC12.SCL, R19.2; no longer R2.1
- net SPI_MISO: now also R19.5; no longer R2.6
- net SPI_MOSI: now also R19.3; no longer R2.4
- net SPI_SCK: now also R19.1; no longer R2.2
- net SPI_SS: now also IC10.IN, R19.8; no longer R3.8
Other:
- moved on the sheet: IC7

Commit message: - replaced LTC3350 with LTC3351, updated schematic and board
Parts:
- removed C10, C11, C12, C16, C17, C18, C19: 0.1μF, rcl:C-EUC0402
- removed C15: 10μF, rcl:C-EUC0402
- removed C20: 4.7n, rcl:C-EUC0402
- removed C21: 1μF, rcl:C-EUC0402
- removed IC1: LM74670QDGKRQ1, LM74670 - Smart Diode Rectifier Controller:LM74670
- removed IC4, IC5: SQJ960EP N-FET, SQJ96XEP - MosFET:SQJ96XEP
- removed JP12: (no value), pinhead:PINHD-1X1
- removed R12, R15, R16: 2.7, rcl:R-EU_R0402
- removed R17, R18, R5: 121, rcl:R-EU_R0402
- removed R6: 88.7k, rcl:R-EU_R0402
- removed R7: 2k, rcl:R-EU_R0402
- removed U$2: SIA456DJ, SIA456DJ-T1-GE3 N-Fet:SIA456DJ
- added C27, C33: 0.1μF, rcl:C-EUC0805
- added C32, C_F: 0.1μF, rcl:C-EUC0402
- added CAP1, CAP2, CAP3, CAP4: 15F, rcl:CPOL-EUE5-8.5
- added C_C: 4.7nF, rcl:C-EUC0402
- added C_CAP1, C_CAP2, C_CAP3, C_CAP4, C_SS: 22μF, rcl:C-EUC0402
- added C_CP5: 1μF, rcl:C-EUC0402
- added C_OUT1-1, C_OUT1-2, C_OUT1-3, C_OUT1-4, C_OUT1-5, C_OUT1-6: 100μF, rcl:C-EUC0402
- added C_OUT2-1, C_OUT2-2: 2.2μF, rcl:C-EUC0402
- added D3: CZRB5349B-HF, zener:ZENER
- added IC13: LM74670QDGKRQ1, LM74670 - Smart Diode Rectifier Controller:LM74670
- added IC14: MCP2561-2, MCP2561-2 - High-Speed CAN Transceiver:MCP2561-2
- added IC15: (no value), TS5A1066 Analogue Switch IC:TS5A1066SOT-23
- added JP6: (no value), pinhead:PINHD-1X2
- added L1: 10μH, rcl:L-EUL1812
- added MN1, MN2, MN3, MN5: (no value), SIA456DJ-T1-GE3 N-Fet:SIA456DJ
- added R2: 2k, rcl:R-EU_R0402
- added R23: 741X083102JP 10k, 74x-1133528 Resistor Array:741X083331JP
- added R25: 330k, rcl:R-EU_R0805
- added R26: 120, rcl:R-EU_R0805
- added R_CAP1, R_CAP2, R_CAP3, R_CAP4, R_CAPRTN: 2.7Ω, rcl:R-EU_R0402
- added R_FB01: 400k, rcl:R-EU_R0402
- added R_FB02: 100k, rcl:R-EU_R0402
- added R_FBC1: 732k, rcl:R-EU_R0402
- added R_FBC2: 274k, rcl:R-EU_R0402
- added R_PF1, R_PF3: 30.1k, rcl:R-EU_R0402
- added R_PF2: 10k, rcl:R-EU_R0402
- added R_SNSC: 0.003Ω, rcl:R-EU_R0402
- added R_SNSI: 0.064Ω, rcl:R-EU_R0402
- added R_T: 88.7k, rcl:R-EU_R0402
- added R_T1: 100k THERM, rcl:R-EU_R0402
- added R_TST: 20Ω, rcl:R-EU_R0402
- C1: value 0.1μF -> 1μF; device rcl:C-EUC0805 -> rcl:C-EUC0402
- C13: value 0.1μF -> 4.7μF
- C3: value 0.1μF -> 4.7nF; device rcl:C-EUC0805 -> rcl:C-EUC0402
- C5: value (none) -> 100pF
- C6: value 4.7n -> 0.1μF
- D1: value CZRB5349B-HF -> (none); device zener:ZENER -> diode:SCHOTTKY-DIODESMC
- IC10: value (none) -> MCP2515; device TS5A1066 Analogue Switch IC:TS5A1066SOT-23 -> MCP2515-I-ML - Standalonce CAN Controller with SPI Interface:MCP2515-I-ML
- IC11: value LM74670QDGKRQ1 -> PRQV8.00CR1510Y00L; device LM74670 - Smart Diode Rectifier Controller:LM74670 -> PRQV8.00CR1510Y00L - 8MHz resonator:PRQV
- IC12: value LTC3350 -> SQJ960EP N-FET; device LTC3350fc High Current Supercapacitor Backup Controller and System Monitor:LTC3350 -> SQJ96XEP - MosFET:SQJ96XEP
- IC16: value SIA456DJ -> (none)
- IC3: value LM74670QDGKRQ1 -> (none); device LM74670 - Smart Diode Rectifier Controller:LM74670 -> LTC3351f - Hot Swappable Supercapacitor Charger, Backup Controller and System Monitor:LTC3351
- IC6: value ATTINY4313-MMH -> LM74670QDGKRQ1; device ATtiny4313 microcontroller:ATTINY4313VQFN-20 -> LM74670 - Smart Diode Rectifier Controller:LM74670
- IC7: value PRQV8.00CR1510Y00L -> ATTINY4313-MMH; device PRQV8.00CR1510Y00L - 8MHz resonator:PRQV -> ATtiny4313 microcontroller:ATTINY4313VQFN-20
- IC8: value MCP2515 -> LM74670QDGKRQ1; device MCP2515-I-ML - Standalonce CAN Controller with SPI Interface:MCP2515-I-ML -> LM74670 - Smart Diode Rectifier Controller:LM74670
- IC9: value MCP2561-2 -> SQJ960EP N-FET; device MCP2561-2 - High-Speed CAN Transceiver:MCP2561-2 -> SQJ96XEP - MosFET:SQJ96XEP
- JP1: value (none) -> JUMPER-SMT_2_NO_SILK; device pinhead:PINHD-1X2 -> SparkFun-Jumpers:JUMPER-SMT_2_NO_SILK
- JP3: value JUMPER-SMT_2_NO_SILK -> (none); device SparkFun-Jumpers:JUMPER-SMT_2_NO_SILK -> pinhead:PINHD-1X2
- JP8: device pinhead:PINHD-1X2 -> pinhead:PINHD-1X1
- R1: value 120 -> 100k; device rcl:R-EU_R0805 -> rcl:R-EU_R0402
- R10, R11: value 2.7 -> 10Ω
- R13, R14: value 2.7 -> 10k
- R3: value 741X083102JP 10k -> 10k; device 74x-1133528 Resistor Array:741X083331JP -> rcl:R-EU_R0402
- R4: value (none) -> 10k
- R8: value 2k -> 10k
- R9: value 330k -> 100Ω; device rcl:R-EU_R0805 -> rcl:R-EU_R0402
- renumbered 6V0 to X2, C14 to C31, C2 to C30, C4 to C34, C8 to C29, C9 to C28, CAN to X1, DYNAMO to J1, IC2 to IC17, JP11 to JP7, R19 to R24, SPI to CONN1, SPLIT to TP1, U$1 to IC16
Connections:
- removed net N$17: C6.2, R7.2
- removed net N$21: IC12.GPI
- removed net N$22: C10.1, IC12.CFP
- removed net N$23: C10.2, IC12.CFN
- removed net N$24: C11.1, IC12.VCAP
- removed net N$25: C11.2, IC12.VCAPP5
- removed net N$26: C12.2, IC12.TGATE
- removed net N$28: C13.1, C15.1, IC12.DRVCC, IC12.INTVCC
- removed net N$29: C16.1, C17.2, R10.2
- removed net N$30: C17.1, C18.2, R11.2
- removed net N$31: C18.1, C19.2, R12.2
- removed net N$32: IC12.CAP1, R10.1
- removed net N$33: IC12.CAP2, R11.1
- removed net N$34: IC12.CAP3, R12.1
- removed net N$35: IC12.CAP4, R13.1
- removed net N$36: C19.1, R13.2, R15.1
- removed net N$37: IC12.CAPRTN, R14.1
- removed net N$38: IC12.CAPFB, R15.2, R16.1
- removed net N$39: IC12.PFI, R17.2, R18.1
- removed net N$40: C20.2, IC12.VIN
- removed net N$41: R17.1
- removed net N$5: JP1.2, JP3.2
- new net BGATE: IC3.BGATE, MN3.G
- new net BST: C6.1, D1.C, IC3.BST
- new net CAP1: IC3.CAP1, R_CAP1.1
- new net CAP2: IC3.CAP2, R_CAP2.1
- new net CAP3: IC3.CAP3, R_CAP3.1
- new net CAP4: IC3.CAP4, R_CAP4.1
- new net CAPFB: IC3.CAPFB, R_FBC1.1, R_FBC2.2
- new net CAPRTN: IC3.CAPRTN, R_CAPRTN.1
- new net CFN: C_F.2, IC3.CFN
- new net CFP: C_F.1, IC3.CFP
- new net CSS: C_SS.2, IC3.CSS
- new net CTIMER: C3.2, IC3.CTIMER
- new net DRVCC: C13.1, C7.1, D1.A, IC3.DRVCC, IC3.INTVCC
- new net GPI: IC3.GPI, R1.2, R_T1.1
- new net ICAP: IC3.ICAP, L1.2, R_SNSC.1
- new net ITST: IC3.ITST, R_TST.1
- new net N$1: IC3.SRC, MN1.S, MN5.S
- new net N$2: MN1.G, R10.1
- new net N$6: IC3.ISNSP_CHG, IC3.ISNSP_HS, MN5.D, R_SNSI.1
- new net N$7: CAP3.+, CAP4.-, R_CAP3.2
- new net N$8: CAP2.+, CAP3.-, R_CAP2.2
- new net OUTFB: C5.2, IC3.OUTFB, R_FB01.2, R_FB02.1
- new net OV: IC3.OV, R_PF2.2, R_PF3.1
- new net RETRYB: IC3.RETRYB, R13.1, R14.1
- new net RT: IC3.RT, R_T.1
- new net SW: C6.2, IC3.SW, L1.1, MN2.S, MN3.D
- new net TGATE: IC3.TGATE, MN2.G
- new net UV: IC3.UV, R_PF1.2, R_PF2.1
- new net VC: IC3.VC, R2.1
- new net VCAP: CAP4.+, C_CAP1.1, C_CAP2.1, C_CAP3.1, C_CAP4.1, C_CP5.1, IC3.VCAP, R_CAP4.2, R_FBC1.2, R_SNSC.2
- new net VCAPP5: C_CP5.2, IC3.VCAPP5
- new net VDD: R3.1, R4.1, R8.1
- new net VIN: MN1.D, R9.2, R_PF1.1
- new net VOUT: C5.1, C_OUT1-1.1, C_OUT1-2.1, C_OUT1-3.1, C_OUT1-4.1, C_OUT1-5.1, C_OUT1-6.1, C_OUT2-1.1, C_OUT2-2.1, C_SS.1, IC3.ISNSM, IC3.VOUT, MN2.D, R14.2, R_FB01.1, R_SNSI.2
- net !PFO!: now also IC3.VINGD, R8.2; no longer IC12.!PFO!
- net !SMBALERT!: now also IC3.!SMBALERT!, IC7.OC0A/PCINT2-PB2, R3.2; no longer IC12.!SMBALERT!, IC6.OC0A/PCINT2-PB2
- net 5V0: now also C32.1, IC10.VDD, IC14.VCC, IC15.VCC, IC7.VCC, R23.1, R23.3, R25.2; no longer C7.1, IC10.VCC, IC6.VCC, IC8.VDD, IC9.VCC, R3.1, R3.3, R9.2
- net CANH: now also IC14.CANH, R26.2; no longer IC9.CANH, R1.2
- net CANL: now also IC14.CANL, R26.1; no longer IC9.CANL, R1.1
- net CAPGD: now also IC3.CAPGD, R4.2; no longer IC12.CAPGD
- net CKOUT: now also IC10.OSC1, IC7.PCINT13/CKOUT/XCK/INT0-PD2; no longer IC6.PCINT13/CKOUT/XCK/INT0-PD2, IC8.OSC1
- net DEBUGWIRE/RESET: now also IC7.!RESET!/DW/PCINT10-PA2; no longer IC6.!RESET!/DW/PCINT10-PA2
- net DYNAMO_1: now also D3.AN, IC6.CATHODE, IC8.ANODE, IC9.D1, IC9.S2; no longer D2.AN, IC1.CATHODE, IC3.ANODE, IC5.D1, IC5.S2
- net DYNAMO_2: now also D2.AN, IC12.D2, IC12.S1, IC13.ANODE; no longer D1.AN, IC11.ANODE, IC4.D2, IC4.S1
- net FET1_G: now also IC6.GATE, IC6.GATE_PULLD, IC9.G1; no longer IC1.GATE, IC1.GATE_PULLD, IC5.G1
- net FET2_G: now also IC8.GATE, IC8.GATE_PULLD, IC9.G2; no longer IC3.GATE, IC3.GATE_PULLD, IC5.G2
- net FET3_G: now also IC12.G1, IC13.GATE, IC13.GATE_PULLD; no longer IC11.GATE, IC11.GATE_PULLD, IC4.G1
- net FET4_G: now also IC12.G2; no longer IC4.G2
- net GND: now also C1.2, C3.1, C32.2, CAP1.-, C_C.2, C_CAP1.2, C_CAP2.2, C_CAP3.2, C_CAP4.2, C_OUT1-1.2, C_OUT1-2.2, C_OUT1-3.2, C_OUT1-4.2, C_OUT1-5.2, C_OUT1-6.2, C_OUT2-1.2, C_OUT2-2.2, IC11.GND, IC12.S2, IC14.GND, IC15.GND, IC3.PGND, IC3.SGND, IC6.ANODE, IC9.S1, JP6.2, MN3.S, R13.2, R_CAPRTN.2, R_FB02.2, R_FBC2.1, R_PF3.2, R_T.2, R_T1.2, R_TST.2; no longer C15.2, C16.2, C20.1, C21.2, IC1.ANODE, IC12.GND, IC12.SGND, IC4.S2, IC5.S1, IC6.GND, IC8.GND, IC9.GND, JP3.1, R14.2, R18.2, R5.2
- net I2C_SDA: now also IC15.COM, IC3.SDA; no longer IC10.COM, IC12.SDA
- net ICSP_DI/MISO: now also IC15.NO, IC7.MOSI/DI/SDA/PCINT5-PB5; no longer IC10.NO, IC6.MOSI/DI/SDA/PCINT5-PB5
- net ICSP_DO/MOSI: now also IC7.MISO/DO/PCINT6-PB6; no longer IC6.MISO/DO/PCINT6-PB6
- net ICSP_SCK: now also IC3.SCL, IC7.USCK/SCL/SCK/PCINT7-PB7; no longer IC12.SCL, IC6.USCK/SCL/SCK/PCINT7-PB7
- net INT1: now also IC10.!INT!, IC7.PCINT14/INT1-PD3; no longer IC6.PCINT14/INT1-PD3, IC8.!INT!
- net N$12: now also C33.1, IC13.VCAPL; no longer C3.1, IC11.VCAPL
- net N$13: now also C33.2, IC13.VCAPH; no longer C3.2, IC11.VCAPH
- net N$14: now also IC8.VCAPL; no longer IC3.VCAPL
- net N$15: now also IC8.VCAPH; no longer IC3.VCAPH
- net N$16: now also CAP1.+, CAP2.-, R_CAP1.2; no longer IC12.ITST, R5.1
- net N$18: now also MN5.G, R11.2; no longer IC12.RT, R6.1
- net N$19: now also C_C.1, R2.2; no longer C6.1, R6.2
- net N$20: now also IC3.HS_GATE, R10.2, R11.1; no longer IC12.VC, R7.1
- net N$27: now also IC3.VIN, R9.1; no longer C12.1, IC12.BST
- net N$3: now also C27.2, IC6.VCAPH; no longer C1.2, IC1.VCAPH
- net N$4: now also JP4.2, JP6.1; no longer JP1.1, JP2.2
- net N$9: now also C27.1, IC6.VCAPL; no longer C1.1, IC1.VCAPL
- net OUT+: now also IC12.D1, IC13.CATHODE, IC8.CATHODE, IC9.D2, JP4.1; no longer IC11.CATHODE, IC3.CATHODE, IC4.D1, IC5.D2, JP2.1
- net RESET: now also IC10.!RESET!, R23.4; no longer IC8.!RESET!, R3.4
- net RXCAN: now also IC10.RXCAN, IC14.RXD; no longer IC8.RXCAN, IC9.RXD
- net SPI_MISO: now also IC10.SO; no longer IC8.SO
- net SPI_MOSI: now also IC10.SI; no longer IC8.SI
- net SPI_SCK: now also IC10.SCK; no longer IC8.SCK
- net SPI_SS: now also IC10.!CS!, IC15.IN, IC7.OC1B/PCINT4-PB4; no longer IC10.IN, IC6.OC1B/PCINT4-PB4, IC8.!CS!
- net SPLIT: now also IC14.SPLIT; no longer IC9.SPLIT
- net STBY: now also IC14.STBY, IC7.AIN1/PCINT1-PB1, R23.2; no longer IC6.AIN1/PCINT1-PB1, IC9.STBY, R3.2
- net TXCAN: now also IC10.TXCAN, IC14.TXD; no longer IC8.TXCAN, IC9.TXD
- net VCC2P5: now also C1.1, IC3.CAP_SLCT0, IC3.CAP_SLCT1, IC3.VCC2P5, R1.1; no longer C21.1, IC12.CAP_SLCT0, IC12.CAP_SLCT1, IC12.VCC2P5
- net XTAL1: now also IC11.XTAL1, IC7.PCINT8/CLKI/XTAL1-PA0; no longer IC6.PCINT8/CLKI/XTAL1-PA0, IC7.XTAL1
- net XTAL2: now also IC11.XTAL2, IC7.PCINT9/XTAL2-PA1; no longer IC6.PCINT9/XTAL2-PA1, IC7.XTAL2
- net ZENER_COMMON: now also D3.CAT; no longer D1.CAT
- net ZERO_CROSS: now also JP8.1, R25.1; no longer JP12.1, R9.1
Other:
- note added: "Overall Concept: LTC3350 shall mirror a normal bicycle dynamo behaviour as close as possible: accept 6V / 3W and give out 6V / 3W in other words: charge the supercaps with max. 500mA, give out 500mA"
- note added: "TODO: Vcap Voltage"
- note added: "TODO: what is Vdd ?"
- note added: "input stage with overvoltage protection to Vzener=18v"
- note added: "p. 23 - Setting Vout Voltage in Backup Mode Vout = ( 1 + (Rfb02/Rfb02) ) * 1.2V with Rfb01 = 400k and Rfb02 = 100k we get: Vout = (1 + 4 ) *1.2 = 6v"
- note added: "p.21"
- note added: "p.21 - Setting Input and Charge Currents Iin = 32mV / Rsnsc <=> 32mV / 500mA = 64mΩ Ipeak = 58mV / 64mΩ = 906mA"
- note added: "p.21 - Setting Input and Charge Currents Iin = 32mV / Rsnsi <=> 32mV / 0.5A = 0.064Ω"
- note added: "p.22 - Power-Fail Comparator Input Voltage Threshold Power-fail condition: Vin_fail = ( 1+ (Rpf1/Rpf2) ) * Vpfi_TH Power-good condition: Vin_good = ( 1+ (Rpf1/Rpf2) ) * (Vpfi_TH + Vpfi_HYS) Vpfi_TH = 1.17V Vpfi_HYS = 30mV with Rpf1 = 30.1 k and Rpfi2 = 10k it gives: Vin_fail = 4.6917V Vin_good = 4.7217V"
- note added: "p.22 - Setting Vcap Voltage Vcap = (1+ (Rfvc1/Rfbc2) ) * CAPFBREF"
- note added: "p.24 - Compensation Rfb01 * Cfb01 = 1 / (2Pi * 2kHz) is equivalent to: Cfb01 = Rfb01 / ( 2Pi * 2kHz ) that gives: Cfb01 = 400kΩ / ( 6.28 * 2000) ="
- note removed: "input statge with overvoltage protection to Vzener=18v"
- moved on the sheet: C1, C13, C3, C5, C6, C7, D2, JP2, JP4, JP5, R1, R10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

Commit message: - continued work on POC board
Parts:
- removed JP2, JP5: JUMPER-SMT_2_NO_SILK, SparkFun-Jumpers:JUMPER-SMT_2_NO_SILK
- removed JP3: (no value), pinhead:PINHD-1X2
- removed TP1: TPB2,54, testpad:TPB2,54
Connections:
- removed net SPLIT: IC14.SPLIT, TP1.TP
- removed net VOUT: C5.1, C_OUT1-1.1, C_OUT1-2.1, C_OUT1-3.1, C_OUT1-4.1, C_OUT1-5.1, C_OUT1-6.1, C_OUT2-1.1, C_OUT2-2.1, C_SS.1, IC3.ISNSM, IC3.VOUT, MN2.D, R14.2, R_FB01.1, R_SNSI.2
- net 6V0: now also C5.1, C_OUT1-1.1, C_OUT1-2.1, C_OUT1-3.1, C_OUT1-4.1, C_OUT1-5.1, C_OUT1-6.1, C_OUT2-1.1, C_OUT2-2.1, C_SS.1, IC3.ISNSM, IC3.VOUT, MN2.D, R14.2, R_FB01.1, R_SNSI.2
- net N$4: now also JP1.1
- net VIN: now also JP1.2
Other:
- moved on the sheet: JP1
