File: eagle design/MJ808 clone - all driver - POC.sch (EAGLE design)
At the start: 28 parts, among them IC1 ATTINY4313-MMH, IC2 PRQV8.00CR1510Y00L, IC3 MCP2515, IC5 MCP2561-2, IC6 MAX16820, IC7 LDK320ADU50R, K1 CRTL, Q1 SiA456DJ, X3 BAT

Commit message: - renamed gerber folder names - replaced SPST-NO tactile pushbutton with actual model used in the prod board
Parts:
- removed K1: CRTL, Seeed-Switch:SMD-SWITCH-TACTILE-SPST-NO(4P-D6.0MM)
- added POWER: TL3305CF260QG, TL3305-844809 SPST-NO Tact Switch:TL3305-844809
- R10: value 0.15 / 1W -> 0.25 / 1W
Connections:
- net 5V0: now also POWER.P$1; no longer K1.B1
- net SWITCH: now also POWER.P$2; no longer K1.A1

Commit message: - replaced oscillator, fet and mj808 utility led with better components, updated schematics - added/removed relevant datasheets for above changes
Parts:
- IC2: value PRQV8.00CR1510Y00L -> PBRC8.00GR50X000
- LED2: value APHBM2012LSURKZGKC -> IN-S85DATRG
- Q1: value SiA456DJ -> SQA470EEJ-T1_GE3
Changed lines of the file:
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@@
 <part name="D1" library="diode" library_urn="urn:adsk.eagle:library:210" deviceset="DIODE-" device="SOD123" package3d_urn="urn:adsk.eagle:package:43420/1" value="PMEG2010ER,115"/>
 <part name="L1" library="SparkFun-Coils" library_urn="urn:adsk.eagle:library:512" deviceset="INDUCTOR" device="-SRN6045-33UH" package3d_urn="urn:adsk.eagle:package:37576/1" value="VLS6045EX-150M-CA - 15uH"/>
-<part name="Q1" library="SIA456DJ-T1-GE3  N-Fet" deviceset="SIA456DJ" device="" value="SiA456DJ"/>
+<part name="Q1" library="SIA456DJ-T1-GE3  N-Fet" deviceset="SIA456DJ" device="" value="SQA470EEJ-T1_GE3"/>
 <part name="IC3" library="MCP2515-I-ML - Standalonce CAN Controller with SPI Interface" deviceset="MCP2515-I-ML" device="" value="MCP2515"/>
 <part name="IC5" library="MCP2561-2 - High-Speed CAN Transceiver" deviceset="MCP2561-2" device="" value="MCP2561-2"/>
@@
 <attribute name="SPICEPREFIX" value="X"/>
 </part>
-<part name="IC2" library="PRQV8.00CR1510Y00L - 8MHz resonator" deviceset="PRQV" device="" value="PRQV8.00CR1510Y00L"/>
+<part name="IC2" library="PRQV8.00CR1510Y00L - 8MHz resonator" deviceset="PRQV" device="" value="PBRC8.00GR50X000"/>
 <part name="R1" library="rcl" library_urn="urn:adsk.eagle:library:334" deviceset="R-EU_" device="R0402" package3d_urn="urn:adsk.eagle:package:23547/2" value="10k"/>
 <part name="LED1" library="con-molex" library_urn="urn:adsk.eagle:library:165" deviceset="22-23-2021" device="" value="LEDXMLBWT-00-0000-0000U20E2 "/>
@@
 <part name="C4" library="rcl" library_urn="urn:adsk.eagle:library:334" deviceset="C-EU" device="C0402" package3d_urn="urn:adsk.eagle:package:23626/1" value="1μF"/>
 <part name="R2" library="rcl" library_urn="urn:adsk.eagle:library:334" deviceset="R-EU_" device="R0402" package3d_urn="urn:adsk.eagle:package:23547/2" value="10k"/>
-<part name="LED2" library="APHBM2012LSURKZGKC" deviceset="APHBM2012LSURKZGKC" device="" value="APHBM2012LSURKZGKC"/>
+<part name="LED2" library="APHBM2012LSURKZGKC" deviceset="APHBM2012LSURKZGKC" device="" value="IN-S85DATRG"/>
 <part name="SPI" library="5034800600 FPC Connector" deviceset="5034800600" device="" value="5034800600"/>
 <part name="SPLIT" library="testpad" library_urn="urn:adsk.eagle:library:385" deviceset="TP" device="B2,54" package3d_urn="urn:adsk.eagle:package:27948/1"/>
