File: eagle design/MJ818 clone - all driver - POC.sch (EAGLE design)
At the start: 37 parts, among them IC1 MAX16839, IC2 ATTINY4313-MMH, IC3 PRQV8.00CR1510Y00L, IC4 LDK320ADU50R, IC5 MCP2515, IC6 MCP2561-2, IC7 MAX16820, Q1 SiA456DJ, X1 CAN, X2 XPERED-L1-R250-00401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

Commit message: - replaced oscillator, fet and mj808 utility led with better components, updated schematics - added/removed relevant datasheets for above changes
Parts:
- IC3: value PRQV8.00CR1510Y00L -> PBRC8.00GR50X000
- LED1, LED2, LED3, LED4, LED5, LED6, LED7, LED8, LED9: device AM2520SURC03-31454 - Red SMD LED:AM2520SURC03-31454 -> 1374-CLM2D-RCC-ACC-1064252 - Red SMD LED:1374-CLM2D-RCC-ACC-1064252
- Q1: value SiA456DJ -> SQA470EEJ-T1_GE3
- R6: value 30R/0.5W -> WSLT2010R2200FEB18 / 0.22Ohm 1W; device rcl:R-EU_R1206 -> rcl:R-EU_R2010
Changed lines of the file:
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@@
 </classes>
 <parts>
-<part name="R6" library="rcl" library_urn="urn:adsk.eagle:library:334" deviceset="R-EU_" device="R1206" package3d_urn="urn:adsk.eagle:package:23540/2" value="30R/0.5W"/>
+<part name="R6" library="rcl" library_urn="urn:adsk.eagle:library:334" deviceset="R-EU_" device="R2010" package3d_urn="urn:adsk.eagle:package:23551/2" value="WSLT2010R2200FEB18 / 0.22Ohm 1W"/>
 <part name="C7" library="rcl" library_urn="urn:adsk.eagle:library:334" deviceset="C-EU" device="C0805" package3d_urn="urn:adsk.eagle:package:23617/2" value="47μF"/>
 <part name="D1" library="diode" library_urn="urn:adsk.eagle:library:210" deviceset="DIODE-" device="SOD123" package3d_urn="urn:adsk.eagle:package:43420/1" value="PMEG2010ER,115"/>
-<part name="Q1" library="SIA456DJ-T1-GE3  N-Fet" deviceset="SIA456DJ" device="" value="SiA456DJ"/>
+<part name="Q1" library="SIA456DJ-T1-GE3  N-Fet" deviceset="SIA456DJ" device="" value="SQA470EEJ-T1_GE3"/>
 <part name="IC5" library="MCP2515-I-ML - Standalonce CAN Controller with SPI Interface" deviceset="MCP2515-I-ML" device="" value="MCP2515"/>
 <part name="IC6" library="MCP2561-2 - High-Speed CAN Transceiver" deviceset="MCP2561-2" device="" value="MCP2561-2"/>
@@
 <attribute name="SPICEPREFIX" value="X"/>
 </part>
-<part name="IC3" library="PRQV8.00CR1510Y00L - 8MHz resonator" deviceset="PRQV" device="" value="PRQV8.00CR1510Y00L"/>
+<part name="IC3" library="PRQV8.00CR1510Y00L - 8MHz resonator" deviceset="PRQV" device="" value="PBRC8.00GR50X000"/>
 <part name="X2" library="con-molex" library_urn="urn:adsk.eagle:library:165" deviceset="22-23-2021" device="" package3d_urn="urn:adsk.eagle:package:8078633/1" value="XPERED-L1-R250-00401"/>
 <part name="C4" library="rcl" library_urn="urn:adsk.eagle:library:334" deviceset="C-EU" device="C0402" package3d_urn="urn:adsk.eagle:package:23626/2" value="1μF"/>
@@
 <part name="SPI" library="5034800600 FPC Connector" deviceset="5034800600" device="" value="5034800600"/>
 <part name="L1" library="DE0604A-778075 - Inductor" deviceset="DE0604A-778075" device="" value="SDE0604A-270M - 27uH"/>
-<part name="LED1" library="AM2520SURC03-31454 - Red SMD LED" deviceset="AM2520SURC03-31454" device="" value="604-AM2520SURC03 "/>
-<part name="LED4" library="AM2520SURC03-31454 - Red SMD LED" deviceset="AM2520SURC03-31454" device="" value="604-AM2520SURC03 "/>
-<part name="LED7" library="AM2520SURC03-31454 - Red SMD LED" deviceset="AM2520SURC03-31454" device="" value="604-AM2520SURC03 "/>
-<part name="LED2" library="AM2520SURC03-31454 - Red SMD LED" deviceset="AM2520SURC03-31454" device="" value="604-AM2520SURC03 "/>
-<part name="LED5" library="AM2520SURC03-31454 - Red SMD LED" deviceset="AM2520SURC03-31454" device="" value="604-AM2520SURC03 "/>
-<part name="LED8" library="AM2520SURC03-31454 - Red SMD LED" deviceset="AM2520SURC03-31454" device="" value="604-AM2520SURC03 "/>
-<part name="LED3" library="AM2520SURC03-31454 - Red SMD LED" deviceset="AM2520SURC03-31454" device="" value="604-AM2520SURC03 "/>
-<part name="LED6" library="AM2520SURC03-31454 - Red SMD LED" deviceset="AM2520SURC03-31454" device="" value="604-AM2520SURC03 "/>
-<part name="LED9" library="AM2520SURC03-31454 - Red SMD LED" deviceset="AM2520SURC03-31454" device="" value="604-AM2520SURC03 "/>
+<part name="LED1" library="1374-CLM2D-RCC-ACC-1064252 - Red SMD LED" deviceset="1374-CLM2D-RCC-ACC-1064252" device="" value="604-AM2520SURC03 "/>
+<part name="LED4" library="1374-CLM2D-RCC-ACC-1064252 - Red SMD LED" deviceset="1374-CLM2D-RCC-ACC-1064252" device="" value="604-AM2520SURC03 "/>
+<part name="LED7" library="1374-CLM2D-RCC-ACC-1064252 - Red SMD LED" deviceset="1374-CLM2D-RCC-ACC-1064252" device="" value="604-AM2520SURC03 "/>
+<part name="LED2" library="1374-CLM2D-RCC-ACC-1064252 - Red SMD LED" deviceset="1374-CLM2D-RCC-ACC-1064252" device="" value="604-AM2520SURC03 "/>
+<part name="LED5" library="1374-CLM2D-RCC-ACC-1064252 - Red SMD LED" deviceset="1374-CLM2D-RCC-ACC-1064252" device="" value="604-AM2520SURC03 "/>
+<part name="LED8" library="1374-CLM2D-RCC-ACC-1064252 - Red SMD LED" deviceset="1374-CLM2D-RCC-ACC-1064252" device="" value="604-AM2520SURC03 "/>
+<part name="LED3" library="1374-CLM2D-RCC-ACC-1064252 - Red SMD LED" deviceset="1374-CLM2D-RCC-ACC-1064252" device="" value="604-AM2520SURC03 "/>
+<part name="LED6" library="1374-CLM2D-RCC-ACC-1064252 - Red SMD LED" deviceset="1374-CLM2D-RCC-ACC-1064252" device="" value="604-AM2520SURC03 "/>
+<part name="LED9" library="1374-CLM2D-RCC-ACC-1064252 - Red SMD LED" deviceset="1374-CLM2D-RCC-ACC-1064252" device="" value="604-AM2520SURC03 "/>
 <part name="IC1" library="MAX16839 LED Driver, constant current" deviceset="MAX16839" device="" value="MAX16839 "/>
 <part name="R2" library="rcl" library_urn="urn:adsk.eagle:library:334" deviceset="R-EU_" device="R0603" package3d_urn="urn:adsk.eagle:package:23555/3" value="10R/0.5W"/>
