File: eagle design/MJ828 - POC.brd (EAGLE design)
At the start: 35 x 35 mm, 34 parts, among them IC1 ATTINY4313-MMH, IC2 PRQV8.00CR1510Y00L, IC3 MCP2515, IC5 MCP2561-2, IC6 LDK320ADU50R, SW1 6x6mm spst-no tact, SW2 6x6mm spst-no tact, X1 CAN, X2 BAT

Commit message: - replaced oscillator, fet and mj808 utility led with better components, updated schematics - added/removed relevant datasheets for above changes
Parts:
- IC2: value PRQV8.00CR1510Y00L -> PBRC8.00GR50X000
- SW1, SW2: value 6x6mm spst-no tact -> TL3305CF160QG
Changed lines of the file:
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@@
 <attribute name="VALUE" x="25.25" y="15.25" size="1" layer="27" font="vector" rot="R90" align="center"/>
 </element>
-<element name="IC2" library="PRQV8.00CR1510Y00L - 8MHz resonator" package="SMT" value="PRQV8.00CR1510Y00L" x="22.5" y="13.5" smashed="yes" rot="MR0">
+<element name="IC2" library="PRQV8.00CR1510Y00L - 8MHz resonator" package="SMT" value="PBRC8.00GR50X000" x="22.5" y="13.5" smashed="yes" rot="MR0">
 <attribute name="NAME" x="22.5" y="10.5" size="1" layer="26" font="vector" rot="MR0" align="center"/>
 </element>
@@
 <attribute name="VALUE" x="11" y="22" size="1" layer="28" font="vector" rot="MR180" align="center"/>
 </element>
-<element name="SW2" library="TL3305-844809 SPST-NO Tact Switch" package="SMD" value="6x6mm spst-no tact" x="13" y="6" smashed="yes">
+<element name="SW2" library="TL3305-844809 SPST-NO Tact Switch" package="SMD" value="TL3305CF160QG" x="13" y="6" smashed="yes">
 <attribute name="NAME" x="13" y="2.5" size="1.27" layer="25" font="vector" align="center"/>
 </element>
-<element name="SW1" library="TL3305-844809 SPST-NO Tact Switch" package="SMD" value="6x6mm spst-no tact" x="22" y="6" smashed="yes">
+<element name="SW1" library="TL3305-844809 SPST-NO Tact Switch" package="SMD" value="TL3305CF160QG" x="22" y="6" smashed="yes">
 <attribute name="NAME" x="22" y="2.5" size="1.27" layer="25" font="vector" align="center"/>
 </element>
