File: eagle design/MJ828 - prod.brd (EAGLE design)
At the start: 28 x 22 mm, 35 parts, among them IC1 ATTINY4313-MMH, IC2 PRQV8.00CR1510Y00L, IC4 MCP2515, IC5 MCP2561-2, SW1 6x6mm spst-no tact, SW2 6x6mm spst-no tact

Commit message: - finishing touches for MJ-828 prod board
Parts:
- BAT+: value (none) -> 8V4 Battery +
- BLUE1, BLUE2, BLUE3, BLUE4, BLUE5: value (none) -> HSMN-C170
- GND: value (none) -> Ground
- GREEN: value (none) -> HSMG-C170
- H: value (none) -> CAN High
- IC3: value (none) -> LDK320M50R
- L: value (none) -> CAN Low
- R5: value 741X083102JP -> 741X083103JP / 10kΩ
- R6: value 741X083331JP -> 741X083331JP / 330Ω
- R9: value 741X083102JP -> 741X083102JP / 1kΩ
- RED: value (none) -> HSMS-C170
- YELLOW: value (none) -> HSMY-C170
- moved R2 9.09 mm to (12.8, 4.75), flipped to the bottom, turned to 270 degrees
- moved R4 8.59 mm to (15.2, 4.75), flipped to the bottom, turned to 270 degrees
- moved R1 6.62 mm to (10.2, 4.75), flipped to the bottom, turned to 270 degrees
- moved C1 6.50 mm to (11.5, 4.75), flipped to the bottom, turned to 270 degrees
- moved R3 6.13 mm to (17.8, 4.75), flipped to the bottom, turned to 270 degrees
- moved C2 6.00 mm to (16.5, 4.75), flipped to the bottom, turned to 270 degrees
- moved R9 0.50 mm to (21.5, 14.5)
- moved SW2 0.50 mm to (18.8, 4.75)
- turned BLUE1 to 90 degrees
- turned YELLOW to 90 degrees
- renumbered LED1 to RED, LED2 to YELLOW, LED3 to BLUE2, LED4 to GREEN, LED5 to BLUE1, LED6 to BLUE3, LED7 to BLUE4, LED8 to BLUE5
Connections:
- net CP1: now also IC1.13; no longer IC1.12
- net CP2: now also IC1.12; no longer IC1.11
- net CP3: now also IC1.11; no longer IC1.10
- net CP4: now also IC1.10; no longer IC1.9
- net STBY: now also IC1.9; no longer IC1.13
Routing:
- net 5V0: track 60.4 -> 46.8 mm
- net SW1: track 17.9 -> 7.47 mm, vias 2 -> 1
- net SW2: track 11.6 -> 5.48 mm, vias 2 -> 1
- net STBY: track 17.3 -> 20.6 mm, vias 1 -> 2
- net CP1: track 27.4 -> 24.3 mm
- net CP2: track 11.2 -> 13.0 mm, vias 1 -> 2
- net D_Y: track 10.9 -> 12.2 mm
- net CP3: track 11.1 -> 10.3 mm, vias 3 -> 2
- net GND: track 2.72 -> 2.22 mm
- net N$5: track 13.4 -> 13.0 mm, vias 2 -> 3
- net N$7: track 4.12 -> 3.75 mm, vias 0 -> 1
- net N$1: track 4.12 -> 3.75 mm, vias 0 -> 1
- net N$11: track 5.74 -> 5.42 mm, vias 1 -> 2

Commit message: - replaced oscillator, fet and mj808 utility led with better components, updated schematics - added/removed relevant datasheets for above changes
Parts:
- IC2: value PRQV8.00CR1510Y00L -> PBRC8.00GR50X000
- SW1, SW2: value 6x6mm spst-no tact -> TL3305CF160QG
Changed lines of the file:
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@@
 <attribute name="VALUE" x="22.25" y="10.25" size="1" layer="27" font="vector" rot="R90" align="center"/>
 </element>
-<element name="IC2" library="PRQV8.00CR1510Y00L - 8MHz resonator" package="SMT" value="PRQV8.00CR1510Y00L" x="19.75" y="10.25" smashed="yes" rot="MR0">
+<element name="IC2" library="PRQV8.00CR1510Y00L - 8MHz resonator" package="SMT" value="PBRC8.00GR50X000" x="19.75" y="10.25" smashed="yes" rot="MR0">
 <attribute name="NAME" x="19.75" y="8.5" size="0.75" layer="26" font="vector" rot="MR0" align="center"/>
 </element>
@@
 <attribute name="VALUE" x="13.75" y="16.25" size="1" layer="28" font="vector" rot="MR180" align="center"/>
 </element>
-<element name="SW1" library="TL3305-844809 SPST-NO Tact Switch" package="SMD" value="6x6mm spst-no tact" x="9.25" y="4.75" smashed="yes">
+<element name="SW1" library="TL3305-844809 SPST-NO Tact Switch" package="SMD" value="TL3305CF160QG" x="9.25" y="4.75" smashed="yes">
 <attribute name="NAME" x="12" y="7.75" size="0.75" layer="25" font="vector" align="center"/>
 </element>
-<element name="SW2" library="TL3305-844809 SPST-NO Tact Switch" package="SMD" value="6x6mm spst-no tact" x="18.75" y="4.75" smashed="yes">
+<element name="SW2" library="TL3305-844809 SPST-NO Tact Switch" package="SMD" value="TL3305CF160QG" x="18.75" y="4.75" smashed="yes">
 <attribute name="NAME" x="16" y="7.75" size="0.75" layer="25" font="vector" align="center"/>
 </element>
