File: eagle design/cos/UI_measurement.brd (EAGLE design)
At the start: 35 x 70 mm, 11 parts, among them IC4 LMP92064SD/NOPB

Commit message: - 1st route of UI measure board
Parts:
- removed C10, C7: 0.1μF, rcl:C0402
- removed C6, C9: 10pF, rcl:C0402
- removed IC4: LMP92064SD/NOPB, LMP92064SD - LMP92064 Precision Low-Side, 125-kSps Simultaneous Sampling Current Sensor and Voltage Monitor With SPI:WS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
- removed R10: 324k, rcl:R0402
- removed R11: 100k, rcl:R0402
- added C1: 1μF, rcl:C0402
- added C2: 10pF, rcl:C0402
- added C3, C5: 0.1μF, rcl:C0402
- added IC1: LMP92064SD/NOPB, LMP92064SD - LMP92064 Precision Low-Side, 125-kSps Simultaneous Sampling Current Sensor and Voltage Monitor With SPI:WS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
- added J1: 61300611121, Headers:61300611121
- added R2: 324k, rcl:R0402
- added R3: 100k, rcl:R0402
- added R4: 10k, rcl:R0402
- added TP4: TPSQPAD1-13, testpad:P1-13
- C4: value 1μF -> 10pF
- moved TP2 44.1 mm to (14.8, 6.73), flipped to the top, turned to 270 degrees
- moved TP1 40.5 mm to (11.8, 6.73), flipped to the top, turned to 270 degrees
- moved R1 19.5 mm to (5.50, 13.2), flipped to the top, turned to 90 degrees
- moved C4 16.0 mm to (14.2, 12.2), turned to 90 degrees
Connections:
- net 5V0: now also C2.1, C3.1, C4.1, C5.1, IC1.8_VDD, IC1.9_VDIG, J1.6, R2.2, R4.2; no longer C10.1, C6.1, C7.1, C9.1, IC4.8_VDD, IC4.9_VDIG, R10.2
- net GND: now also J1.1, R3.1; no longer R11.1
- net GND_VIA_INCP: now also C1.2, C2.2, C3.2, C5.2, IC1.10_DGND, IC1.16_RESET, IC1.2_REFG, IC1.3_INCP, IC1.6_INVG, IC1.7_GND, IC1.GND1, TP4.TP; no longer C10.2, C6.2, C7.2, C9.2, IC4.10_DGND, IC4.16_RESET, IC4.2_REFG, IC4.3_INCP, IC4.6_INVG, IC4.7_GND, IC4.GND1
- net INCN: now also IC1.4_INCN; no longer IC4.4_INCN
- net INVP: now also IC1.5_INVP, R2.1, R3.2; no longer IC4.5_INVP, R10.1, R11.2
- net N$17: now also C1.1, IC1.1_REFC; no longer C4.1, IC4.1_REFC
- net SPI_MISO: now also IC1.11_SDO, J1.2; no longer IC4.11_SDO
- net SPI_MOSI: now also IC1.12_SDI, J1.3; no longer IC4.12_SDI
- net SPI_SCK: now also IC1.13_SCLK, J1.4; no longer IC4.13_SCLK
- net SPI_SS_LMP92064SD: now also IC1.14_CSB, J1.5, R4.1; no longer IC4.14_CSB
Routing:
- net 5V0: track 6.86 -> 23.4 mm
- net GND: track 0.25 -> 11.8 mm, vias 1 -> 0
- net SPI_SS_LMP92064SD: track 1.20 -> 8.43 mm
- net INCN: track 32.2 -> 26.7 mm
- net SPI_MISO: track 1.20 -> 6.16 mm, vias 1 -> 0
- net SPI_SCK: track 1.45 -> 4.28 mm, vias 1 -> 0
- net SPI_MOSI: track 1.45 -> 4.03 mm, vias 1 -> 0
- net INVP: track 5.91 -> 8.43 mm
- net N$17: track 1.45 -> 3.55 mm
- net GND_VIA_INCP: vias 8 -> 7
- added copper zone on layer 1, net GND_VIA_INCP
- added copper zone on layer 16, net GND_VIA_INCP
Other:
- board size 35 x 70 mm -> 24 x 26 mm

Commit message: HW rev.1 specified BOM, ERC & DRC check out ok, created gerbers
Parts:
- renumbered TP4 to LOAD
Routing:
- net SPI_MISO: track 6.16 -> 4.87 mm
Other:
- board text added: "5V0"
- board text added: "LMP92064SD breakout"
- board text added: "MISO"
- board text added: "MOSI"
- board text added: "SCK"
- board text added: "SS"
- board text added: "ejovrh rev.1"
- board text added: "high side"
- board text added: "low side"
- board text removed: "vGND"
Changed lines of the file:
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@@
 <wire x1="10.85" y1="5.73" x2="15.85" y2="5.73" width="0.5" layer="21"/>
 <text x="8.35" y="6.73" size="0.75" layer="21" font="vector" rot="R180" align="center-right">TP7</text>
-<text x="21" y="10.5" size="1" layer="29" font="vector" ratio="10" rot="R180" align="center-right">GND</text>
-<text x="18" y="10.5" size="1" layer="29" font="vector" ratio="10" align="center-right">vGND</text>
 <polygon width="0.25" layer="41">
 <vertex x="11" y="13.5"/>
@@
 <vertex x="11" y="13"/>
 </polygon>
+<text x="8.75" y="19.5" size="0.75" layer="21" font="vector" align="center">low side</text>
+<text x="18" y="21.5" size="0.75" layer="21" font="vector" align="center">5V0</text>
+<text x="20.25" y="9.25" size="0.75" layer="21" font="vector" rot="R90" align="center">MISO</text>
+<text x="20.25" y="11.75" size="0.75" layer="21" font="vector" rot="R90" align="center">MOSI</text>
+<text x="20.25" y="14.25" size="0.75" layer="21" font="vector" rot="R90" align="center">SCK</text>
+<text x="20.25" y="17" size="0.75" layer="21" font="vector" rot="R90" align="center">SS</text>
+<text x="18.25" y="4.5" size="0.75" layer="21" font="vector" align="center">GND</text>
+<text x="14.25" y="19.5" size="0.75" layer="21" font="vector" align="center">high side</text>
+<text x="11.75" y="4.25" size="0.75" layer="22" font="vector" rot="MR0" align="center">ejovrh rev.1</text>
+<text x="9.5" y="3.5" size="0.75" layer="21" font="vector" align="center">LMP92064SD breakout</text>
+<wire x1="3.5" y1="22.75" x2="19.5" y2="22.75" width="0.25" layer="21"/>
+<wire x1="19.5" y1="22.75" x2="19.5" y2="18" width="0.25" layer="21"/>
+<wire x1="19.5" y1="18" x2="3.5" y2="18" width="0.25" layer="21"/>
+<wire x1="3.5" y1="18" x2="3.5" y2="22.75" width="0.25" layer="21"/>
 </plain>
 <attributes>
@@
 <elements>
 <element name="IC1" library="LMP92064SD - LMP92064 Precision Low-Side, 125-kSps Simultaneous Sampling Current Sensor and Voltage Monitor With SPI" package="WSON-16" value="LMP92064SD/NOPB" x="12.5" y="12.75" smashed="yes" rot="R270">
-<attribute name="NAME" x="12.5" y="9.5" size="0.75" layer="25" font="vector" align="center"/>
+<attribute name="NAME" x="12.5" y="16" size="0.75" layer="25" font="vector" align="center"/>
 <attribute name="VALUE" x="9.25" y="12.75" size="1" layer="27" font="vector" rot="R270" align="center"/>
 </element>
@@
 <attribute name="MANUFACTURER" value="Wurth Electronics Inc." x="18.13" y="13.05" size="1.778" layer="27" rot="R90" display="off"/>
 <attribute name="MPN" value="61300611121" x="18.13" y="13.05" size="1.778" layer="27" rot="R90" display="off"/>
-<attribute name="NAME" x="16.38" y="9.8" size="1.27" layer="25" rot="R90"/>
 <attribute name="VALUE" x="21.13" y="9.8" size="1.27" layer="27" rot="R90"/>
 </element>
@@
 <attribute name="VALUE" x="17.845" y="17.615" size="1.27" layer="28" rot="MR90"/>
 </element>
-<element name="TP4" library="testpad" library_urn="urn:adsk.eagle:library:385" package="P1-13" package3d_urn="urn:adsk.eagle:package:27946/1" value="TPSQPAD1-13" x="5.43" y="19.4" smashed="yes">
-<attribute name="NAME" x="4.414" y="20.67" size="1.27" layer="25" ratio="10"/>
+<element name="LOAD" library="testpad" library_urn="urn:adsk.eagle:library:385" package="P1-13" package3d_urn="urn:adsk.eagle:package:27946/1" value="TPSQPAD1-13" x="5.43" y="19.4" smashed="yes">
+<attribute name="NAME" x="5.5" y="21.25" size="0.75" layer="25" font="vector" ratio="10" align="center"/>
 <attribute name="POPULARITY" value="0" x="5.43" y="19.4" size="1.778" layer="27" display="off"/>
 <attribute name="TP_SIGNAL_NAME" value="" x="5.43" y="19.4" size="1.778" layer="27" display="off"/>
@@
 <contactref element="IC1" pad="11_SDO"/>
 <contactref element="J1" pad="2"/>
-<wire x1="16.19" y1="12" x2="16.75" y2="11.44" width="0.25" layer="1"/>
-<wire x1="18.13" y1="9.24" x2="16.75" y2="9.24" width="0.25" layer="1"/>
-<wire x1="16.75" y1="11.44" x2="16.75" y2="9.24" width="0.25" layer="1"/>
-<wire x1="16.19" y1="12" x2="14.4" y2="12" width="0.25" layer="1"/>
+<wire x1="15.37" y1="12" x2="18.13" y2="9.24" width="0.25" layer="1"/>
+<wire x1="15.37" y1="12" x2="14.4" y2="12" width="0.25" layer="1"/>
 </signal>
 <signal name="SPI_SCK" class="3">
@@
 <wire x1="18.13" y1="16.86" x2="17.3" y2="16.86" width="0.25" layer="1"/>
 <wire x1="17.3" y1="16.86" x2="16.75" y2="16.31" width="0.25" layer="1"/>
-<wire x1="16.75" y1="16.31" x2="16.75" y2="14.06" width="0.25" layer="1"/>
-<wire x1="16.75" y1="14.06" x2="16.19" y2="13.5" width="0.25" layer="1"/>
-<wire x1="16.19" y1="13.5" x2="14.4" y2="13.5" width="0.25" layer="1"/>
+<wire x1="16.75" y1="16.31" x2="16.75" y2="14.81" width="0.25" layer="1"/>
+<wire x1="16.75" y1="14.81" x2="15.44" y2="13.5" width="0.25" layer="1"/>
+<wire x1="15.44" y1="13.5" x2="14.4" y2="13.5" width="0.25" layer="1"/>
 <wire x1="18.13" y1="16.86" x2="18.86" y2="16.86" width="0.5" layer="16"/>
 <wire x1="19.75" y1="17.75" x2="18.86" y2="16.86" width="0.5" layer="16"/>
@@
 <wire x1="5.5" y1="13.5" x2="5.5" y2="15.75" width="0.25" layer="1"/>
 <wire x1="5.5" y1="16.75" x2="5.5" y2="15.75" width="0.25" layer="1"/>
-<contactref element="TP4" pad="TP"/>
+<contactref element="LOAD" pad="TP"/>
 <polygon width="0.25" layer="1" isolate="0.3">
 <vertex x="0" y="26"/>
