File: eagle design/cos/UI_measurement.sch (EAGLE design)
At the start: 11 parts, among them IC4 LMP92064SD/NOPB

Commit message: - 1st route of UI measure board
Parts:
- removed C9: 10pF, rcl:C-EUC0402
- added C1: 1μF, rcl:C-EUC0402
- added J1: 61300611121, Headers:61300611121
- added R4: 10k, rcl:R-EU_R0402
- added TP4: TPSQPAD1-13, testpad:TPSQPAD1-13
- C4: value 1μF -> 10pF
- renumbered C10 to C5, C6 to C2, C7 to C3, IC4 to IC1, R10 to R2, R11 to R3
Connections:
- net 5V0: now also C4.1, J1.6, R4.2; no longer C9.1
- net GND: now also J1.1
- net GND_VIA_INCP: now also C1.2, TP4.TP; no longer C9.2
- net N$17: now also C1.1; no longer C4.1
- net SPI_MISO: now also J1.2
- net SPI_MOSI: now also J1.3
- net SPI_SCK: now also J1.4
- net SPI_SS_LMP92064SD: now also J1.5, R4.1
Other:
- moved on the sheet: C4

Commit message: HW rev.1 specified BOM, ERC & DRC check out ok, created gerbers
Parts:
- removed TP4: TPSQPAD1-13, testpad:TPSQPAD1-13
- added LOAD: TPSQPAD1-13, testpad:TPSQPAD1-13
Connections:
- net GND_VIA_INCP: now also LOAD.TP; no longer TP4.TP
Other:
- note added: "TP1"
- note added: "Voltage/Current Measurement via SPI device"
- note added: "conceptual overview"
- note added: "technical schematic"
- note removed: "AC Rectifier"
- note removed: "Capacitor switches"
- note removed: "Dynamo Connector & Overvoltage Protection Diodes"
- note removed: "Load"
- note removed: "SPI controlled voltage/current measurement"
- note removed: "rectifier w. zero cross comparator"
- moved on the sheet: C1, C2, C3, C4, C5, IC1, J1, R1, R2, R3, R4, TP1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
