File: eagle design/cos/BQ25798.brd (EAGLE design)
At the start: 160 x 100 mm, 39 parts, among them IC1 PQ25798RQMT, Q1 SPW47N60S5, Q2 SPW47N60S5, Q3 SPW47N60S5, Q4 SPW47N60S5

Commit message: - in library corrected QON to input - specified passives according to datasheet - added N-FET, power inductor, zener diode, USB C connector (both datasheets and libraries), connected accordingly in sch
Parts:
- removed Q1, Q2, Q3, Q4: SPW47N60S5, transistor-fet:P-TO247
- removed Q5: (no value), transistor-fet:P-TO247
- added IC2, IC3, IC4, IC6: CSD17581Q3A, CSD17581Q3A - N-MosFET:PQFN-12
- added IC5: PQ25798RQMT, BQ25798 - Battery Charger:QFN29
- added R10: 100R, rcl:R0805
- added R11: 103AT-2 10k NTC, rcl:R0805
- added R9: 33.01k, rcl:R0805
- added USB-C1: UJ31-CH-G2-SMT-TR, UJ31-CH-G2-SMT-TR - USB C Jack:UJ31CHG2SMTTR
- C1, C4, C5, C8: device rcl:C0805 -> rcl:C0402
- C10: value 10u -> 4.7n/50V
- C11, C14, C15, C16, C17, C18, C19, C2, C3, C9: value 10u -> 10u/50V; device rcl:C0805 -> rcl:C1206
- C12: value 0.1u -> 10u/50V; device rcl:C0805 -> rcl:C1206
- C13: value 10u -> 0.1u; device rcl:C0805 -> rcl:C0402
- C20: value 4.7n -> 10u/50V; device rcl:C0805 -> rcl:C1206
- C7: value 47n -> 47n/50V
- D1, D2: value (none) -> BZT52C2V0T; device diode:SMB -> BZT52C2V0T - Zener diode:SOD-523-2
- IC1: value PQ25798RQMT -> CSD17581Q3A; device BQ25798 - Battery Charger:QFN29 -> CSD17581Q3A - N-MosFET:PQFN-12
- L1: value 1u -> 2.2u/74437346022; device rcl:L2012C -> 74437346022 - Power Inductor:SMD
- R2: value 6.04k -> 10k
- R3: value 100k -> 10k
- R4: value 127k -> 8.2k,0.1%
- R5: value 5.24k -> 10k
- R6: value 33.01k -> 100k
- R7: value k -> 127k
- R8: value 10k -> 5.24k
- moved R5 269.5 mm to (-94.0, -271.8)
- moved L1 246.9 mm to (-101.6, -269.2)
- moved R3 218.2 mm to (-94.0, -259.1)
- moved R8 215.8 mm to (-11.4, -15.2)
- moved R2 150.4 mm to (-94.0, -189.2)
- moved C16 135.9 mm to (-11.4, -119.4)
- moved IC1 130.1 mm to (-55.9, -111.8)
- moved C12 83.3 mm to (-94.0, -182.9)
- moved R1 76.2 mm to (-94.0, -265.4)
- moved C10 76.2 mm to (-94.0, -252.7)
- moved R7 74.9 mm to (-11.4, -50.8)
- moved R6 48.3 mm to (-11.4, -57.1)
- moved C13 25.2 mm to (-27.9, -132.1)
- moved R4 12.7 mm to (-11.4, -63.5)
- moved C11 6.35 mm to (-94.0, -176.5)
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Connections:
- removed net ADAPTER: C5.1, IC1.9, IC1.9_VAC1, Q2.2
- new net B5: USB-C1.B5
- new net V_USB: C5.1, IC2.5_D, IC2.6_D, IC2.7_D, IC2.8_D, IC2.9_D, IC5.9, IC5.9_VAC1, USB-C1.A4, USB-C1.A9, USB-C1.B4, USB-C1.B9
- net !CE!: now also IC5.13_!CE!; no longer IC1.13_!CE!
- net !INT!: now also IC5.21_!INT!; no longer IC1.21_!INT!
- net !QON!: now also IC5.12_!QON!; no longer IC1.12_!QON!
- net 5V0: now also R2.2; no longer R1.1
- net BAT: now also IC5.22_BAT, IC5.23_BAT, IC6.1_S, IC6.2_S, IC6.3_S; no longer IC1.22_BAT, IC1.23_BAT, Q5.3
- net BATP: now also IC5.18_BATP, R10.1; no longer IC1.18_BATP, R7.1
- net BATTERY_PLUS: now also C16.1, IC6.5_D, IC6.6_D, IC6.7_D, IC6.8_D, IC6.9_D, R10.2; no longer C13.1, Q5.2, R7.2
- net BTST1: now also IC5.4_BTST1; no longer IC1.4_BTST1
- net BTST2: now also IC5.19_BTST2; no longer IC1.19_BTST2
- net D+: now also IC5.6_D+, USB-C1.A6, USB-C1.B6; no longer IC1.6_D+
- net D-: now also IC5.7_D-, USB-C1.A7, USB-C1.B7; no longer IC1.7_D-
- net GND: now also C10.1, C20.2, IC5.27_GND, R11.2, R4.1, R6.1, R9.2, USB-C1.A1, USB-C1.A12, USB-C1.B1, USB-C1.B12, USB-C1.S1, USB-C1.S2, USB-C1.S3, USB-C1.S4; no longer C10.2, C20.1, IC1.27_GND, R2.1, R3.1, R6.2, R8.2
- net ILIM_HIZ: now also IC5.17_ILIM_HIZ, R6.2, R7.1; no longer IC1.17_ILIM_HIZ, R3.2, R4.1
- net N$2: now also IC2.1_S, IC2.2_S, IC2.3_S, IC4.1_S, IC4.2_S, IC4.3_S; no longer Q2.3, Q4.3
- net N$3: now also IC1.1_S, IC1.2_S, IC1.3_S, IC3.1_S, IC3.2_S, IC3.3_S; no longer Q1.3, Q3.3
- net N$4: now also IC1.4_G, IC3.4_G, IC5.10_ACDRV2; no longer IC1.10_ACDRV2, Q1.1, Q3.1
- net N$5: now also IC2.4_G, IC4.4_G, IC5.11_ACDRV1; no longer IC1.11_ACDRV1, Q2.1, Q4.1
- net PMID: now also C12.1, IC5.29_PMID; no longer C10.1, IC1.29_PMID
- net PROG: now also IC5.20_PROG, R4.2; no longer IC1.20_PROG, R2.2
- net REGN: now also C10.2, IC5.5_REGN, R7.2, R8.1; no longer C20.2, IC1.5_REGN, R4.2, R5.1
- net SCL: now also IC5.14_SCL; no longer IC1.14_SCL
- net SDA: now also IC5.15_SDA; no longer IC1.15_SDA
- net SDRV: now also IC5.24, IC5.24_SDRV, IC6.4_G; no longer IC1.24, IC1.24_SDRV, Q5.1
- net SOLAR: now also IC1.5_D, IC1.6_D, IC1.7_D, IC1.8_D, IC1.9_D, IC5.8_VAC2; no longer IC1.8_VAC2, Q1.2
- net STAT: now also IC5.1, IC5.1_STAT, R2.1; no longer IC1.1, IC1.1_STAT, R1.2
- net SW1: now also IC5.28_SW1, L1.P$2; no longer IC1.28_SW1, L1.1
- net SW2: now also IC5.26_SW2, L1.P$1; no longer IC1.26_SW2, L1.2
- net SYS: now also C13.1, C20.1, IC5.25_SYS; no longer C12.1, C16.1, IC1.25_SYS
- net TS: now also IC5.16, IC5.16_TS, R11.1, R8.2, R9.1; no longer IC1.16, IC1.16_TS, R5.2, R6.1, R8.1
- net VBUS: now also IC3.5_D, IC3.6_D, IC3.7_D, IC3.8_D, IC3.9_D, IC4.5_D, IC4.6_D, IC4.7_D, IC4.8_D, IC4.9_D, IC5.2_VBUS, IC5.3_VBUS; no longer IC1.2_VBUS, IC1.3_VBUS, Q3.2, Q4.2

Commit message: - added pull-up resistors to the I2C bus and to stat and int signal lines
Parts:
- removed R5: 10k, rcl:R0805
- added R12: 10k, rcl:R0805
- R2: value 10k -> 8.2k,0.1%
- R4: value 8.2k,0.1% -> 10k
- moved R4 262.1 mm to (-104.1, -308.6)
- moved R2 150.4 mm to (-11.4, -63.5)
- moved R3 44.4 mm to (-104.1, -302.3)
- moved R1 32.1 mm to (-104.1, -295.9)
Connections:
- net !INT!: now also R1.1
- net 5V0: now also R1.2, R12.2, R3.2, R4.2; no longer R2.2
- net GND: now also R2.1; no longer R4.1
- net PROG: now also R2.2; no longer R4.2
- net SCL: now also R4.1
- net SDA: now also R3.1
- net STAT: now also R12.1; no longer R2.1
Changed lines of the file:
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@@
 <attribute name="VALUE" x="-12.065" y="-59.69" size="1.27" layer="27"/>
 </element>
-<element name="R4" library="rcl" library_urn="urn:adsk.eagle:library:334" package="R0805" package3d_urn="urn:adsk.eagle:package:23553/2" value="8.2k,0.1% " x="-11.43" y="-63.5" smashed="yes">
+<element name="R2" library="rcl" library_urn="urn:adsk.eagle:library:334" package="R0805" package3d_urn="urn:adsk.eagle:package:23553/2" value="8.2k,0.1% " x="-11.43" y="-63.5" smashed="yes">
 <attribute name="MOUSER" value="667-ERJ-PB6B8201V" x="-11.43" y="-63.5" size="1.778" layer="27" display="off"/>
 <attribute name="NAME" x="-12.065" y="-62.23" size="1.27" layer="25"/>
@@
 <attribute name="VALUE" x="-95.25" y="-185.42" size="1.27" layer="27"/>
 </element>
-<element name="R2" library="rcl" library_urn="urn:adsk.eagle:library:334" package="R0805" package3d_urn="urn:adsk.eagle:package:23553/2" value="10k" x="-93.98" y="-189.23" smashed="yes">
-<attribute name="NAME" x="-94.615" y="-187.96" size="1.27" layer="25"/>
-<attribute name="POPULARITY" value="86" x="-93.98" y="-189.23" size="1.778" layer="27" display="off"/>
-<attribute name="SPICEPREFIX" value="R" x="-93.98" y="-189.23" size="1.778" layer="27" display="off"/>
-<attribute name="VALUE" x="-94.615" y="-191.77" size="1.27" layer="27"/>
-</element>
 <element name="C1" library="rcl" library_urn="urn:adsk.eagle:library:334" package="C0402" package3d_urn="urn:adsk.eagle:package:23626/2" value="0.1u" x="-93.98" y="-195.58" smashed="yes">
 <attribute name="NAME" x="-95.25" y="-194.31" size="1.27" layer="25"/>
@@
 <attribute name="SPICEPREFIX" value="C" x="-93.98" y="-252.73" size="1.778" layer="27" display="off"/>
 <attribute name="VALUE" x="-95.25" y="-255.27" size="1.27" layer="27"/>
-</element>
-<element name="R3" library="rcl" library_urn="urn:adsk.eagle:library:334" package="R0805" package3d_urn="urn:adsk.eagle:package:23553/2" value="10k" x="-93.98" y="-259.08" smashed="yes">
-<attribute name="NAME" x="-94.615" y="-257.81" size="1.27" layer="25"/>
-<attribute name="POPULARITY" value="86" x="-93.98" y="-259.08" size="1.778" layer="27" display="off"/>
-<attribute name="SPICEPREFIX" value="R" x="-93.98" y="-259.08" size="1.778" layer="27" display="off"/>
-<attribute name="VALUE" x="-94.615" y="-261.62" size="1.27" layer="27"/>
-</element>
-<element name="R1" library="rcl" library_urn="urn:adsk.eagle:library:334" package="R0805" package3d_urn="urn:adsk.eagle:package:23553/2" value="10k" x="-93.98" y="-265.43" smashed="yes">
-<attribute name="NAME" x="-94.615" y="-264.16" size="1.27" layer="25"/>
-<attribute name="POPULARITY" value="86" x="-93.98" y="-265.43" size="1.778" layer="27" display="off"/>
-<attribute name="SPICEPREFIX" value="R" x="-93.98" y="-265.43" size="1.778" layer="27" display="off"/>
-<attribute name="VALUE" x="-94.615" y="-267.97" size="1.27" layer="27"/>
-</element>
-<element name="R5" library="rcl" library_urn="urn:adsk.eagle:library:334" package="R0805" package3d_urn="urn:adsk.eagle:package:23553/2" value="10k" x="-93.98" y="-271.78" smashed="yes">
-<attribute name="NAME" x="-94.615" y="-270.51" size="1.27" layer="25"/>
-<attribute name="POPULARITY" value="86" x="-93.98" y="-271.78" size="1.778" layer="27" display="off"/>
-<attribute name="SPICEPREFIX" value="R" x="-93.98" y="-271.78" size="1.778" layer="27" display="off"/>
-<attribute name="VALUE" x="-94.615" y="-274.32" size="1.27" layer="27"/>
 </element>
 <element name="L1" library="74437346022 - Power Inductor" package="SMD" value="2.2u/74437346022" x="-101.6" y="-269.24" smashed="yes">
@@
 <attribute name="NAME" x="-105.56" y="-278.94" size="0.75" layer="25" font="vector" rot="R90" align="center"/>
 <attribute name="VALUE" x="-92.56" y="-278.94" size="0.75" layer="27" font="vector" rot="R90" align="center"/>
+</element>
+<element name="R12" library="rcl" library_urn="urn:adsk.eagle:library:334" package="R0805" package3d_urn="urn:adsk.eagle:package:23553/2" value="10k" x="-104.14" y="-289.56" smashed="yes">
+<attribute name="NAME" x="-104.775" y="-288.29" size="1.27" layer="25"/>
+<attribute name="POPULARITY" value="86" x="-104.14" y="-289.56" size="1.778" layer="27" display="off"/>
+<attribute name="SPICEPREFIX" value="R" x="-104.14" y="-289.56" size="1.778" layer="27" display="off"/>
+<attribute name="VALUE" x="-104.775" y="-292.1" size="1.27" layer="27"/>
+</element>
+<element name="R1" library="rcl" library_urn="urn:adsk.eagle:library:334" package="R0805" package3d_urn="urn:adsk.eagle:package:23553/2" value="10k" x="-104.14" y="-295.91" smashed="yes">
+<attribute name="NAME" x="-104.775" y="-294.64" size="1.27" layer="25"/>
+<attribute name="POPULARITY" value="86" x="-104.14" y="-295.91" size="1.778" layer="27" display="off"/>
+<attribute name="SPICEPREFIX" value="R" x="-104.14" y="-295.91" size="1.778" layer="27" display="off"/>
+<attribute name="VALUE" x="-104.775" y="-298.45" size="1.27" layer="27"/>
+</element>
+<element name="R3" library="rcl" library_urn="urn:adsk.eagle:library:334" package="R0805" package3d_urn="urn:adsk.eagle:package:23553/2" value="10k" x="-104.14" y="-302.26" smashed="yes">
+<attribute name="NAME" x="-104.775" y="-300.99" size="1.27" layer="25"/>
+<attribute name="POPULARITY" value="86" x="-104.14" y="-302.26" size="1.778" layer="27" display="off"/>
+<attribute name="SPICEPREFIX" value="R" x="-104.14" y="-302.26" size="1.778" layer="27" display="off"/>
+<attribute name="VALUE" x="-104.775" y="-304.8" size="1.27" layer="27"/>
+</element>
+<element name="R4" library="rcl" library_urn="urn:adsk.eagle:library:334" package="R0805" package3d_urn="urn:adsk.eagle:package:23553/2" value="10k" x="-104.14" y="-308.61" smashed="yes">
+<attribute name="NAME" x="-104.775" y="-307.34" size="1.27" layer="25"/>
+<attribute name="POPULARITY" value="86" x="-104.14" y="-308.61" size="1.778" layer="27" display="off"/>
+<attribute name="SPICEPREFIX" value="R" x="-104.14" y="-308.61" size="1.778" layer="27" display="off"/>
+<attribute name="VALUE" x="-104.775" y="-311.15" size="1.27" layer="27"/>
 </element>
 </elements>
@@
 <contactref element="IC5" pad="1_STAT"/>
 <contactref element="IC5" pad="1"/>
-<contactref element="R2" pad="1"/>
-<wire x1="2.085" y1="5.41" x2="-94.93" y2="-189.23" width="0" layer="19" extent="1-1"/>
+<contactref element="R12" pad="1"/>
+<wire x1="2.085" y1="5.41" x2="-105.09" y2="-289.56" width="0" layer="19" extent="1-1"/>
 <wire x1="2.46" y1="5.71" x2="2.085" y2="5.41" width="0" layer="19" extent="1-1"/>
 </signal>
@@
 <signal name="!INT!">
 <contactref element="IC5" pad="21_!INT!"/>
+<contactref element="R1" pad="1"/>
+<wire x1="5.71" y1="4.21" x2="-105.09" y2="-295.91" width="0" layer="19" extent="1-1"/>
 </signal>
 <signal name="!QON!">
@@
 <signal name="SDA">
 <contactref element="IC5" pad="15_SDA"/>
+<contactref element="R3" pad="1"/>
+<wire x1="4.81" y1="1.91" x2="-105.09" y2="-302.26" width="0" layer="19" extent="1-1"/>
 </signal>
 <signal name="SCL">
 <contactref element="IC5" pad="14_SCL"/>
+<contactref element="R4" pad="1"/>
+<wire x1="4.41" y1="1.91" x2="-105.09" y2="-308.61" width="0" layer="19" extent="1-1"/>
 </signal>
 <signal name="GND">
 <contactref element="R9" pad="2"/>
 <contactref element="R6" pad="1"/>
-<contactref element="R4" pad="1"/>
+<contactref element="R2" pad="1"/>
 <contactref element="G2" pad="-"/>
 <contactref element="C14" pad="2"/>
@@
 </signal>
 <signal name="PROG">
-<contactref element="R4" pad="2"/>
+<contactref element="R2" pad="2"/>
 <contactref element="IC5" pad="20_PROG"/>
 <wire x1="5.71" y1="3.81" x2="-10.48" y2="-63.5" width="0" layer="19" extent="1-1"/>
@@
 </signal>
 <signal name="5V0">
-<contactref element="R2" pad="2"/>
+<contactref element="R12" pad="2"/>
+<contactref element="R1" pad="2"/>
+<contactref element="R4" pad="2"/>
+<contactref element="R3" pad="2"/>
+<wire x1="-103.19" y1="-302.26" x2="-103.19" y2="-308.61" width="0" layer="19" extent="1-1"/>
+<wire x1="-103.19" y1="-295.91" x2="-103.19" y2="-302.26" width="0" layer="19" extent="1-1"/>
+<wire x1="-103.19" y1="-289.56" x2="-103.19" y2="-295.91" width="0" layer="19" extent="1-1"/>
 </signal>
 <signal name="B5">

Commit message: - defined netclasses & associated named nets to classes
Parts:
- removed R12: 10k, rcl:R0805
- added R5: 8.2k,0.1%, rcl:R0805
- R2: value 8.2k,0.1% -> 10k
- moved R2 256.1 mm to (-104.1, -302.3)
- moved R3 12.7 mm to (-104.1, -289.6)
Connections:
- net N$2 renamed VAC1_SOURCE
- net N$3 renamed VAC2_SOURCE
- net N$4 renamed ACDRV2
- net N$5 renamed ACDRV1
- net 5V0: now also R2.2; no longer R12.2
- net GND: now also R5.1; no longer R2.1
- net PROG: now also R5.2; no longer R2.2
- net SDA: now also R2.1; no longer R3.1
- net STAT: now also R3.1; no longer R12.1

Commit message: USB 3 version - aligned footprints and names to grid - removed USB-C
Parts:
- removed G1, G2: SL-150-1/2AA/PT, battery:SL-150-1/2AA/PT
- removed USB-C1: UJ31-CH-G2-SMT-TR, UJ31-CH-G2-SMT-TR - USB C Jack:UJ31CHG2SMTTR
- added BATT1, BATT2: (no value), Battery:TH
- R3: value 10k -> 8.2k,0.1%
- R5: value 8.2k,0.1% -> 10k
- moved R3 296.1 mm to (-35.5, -1.50)
- moved R11 227.2 mm to (32.0, -25.5), turned to 270 degrees
- moved C4 215.0 mm to (-85.0, 51.0), turned to 90 degrees
- moved C5 209.8 mm to (-59.5, 49.5), turned to 90 degrees
- moved C19 207.4 mm to (35.5, -78.0)
- moved C18 207.1 mm to (35.5, -72.0)
- moved C15 207.0 mm to (35.5, -59.5)
- moved C20 206.9 mm to (35.5, -85.0)
- moved C17 206.9 mm to (35.5, -66.0)
- moved D1 204.0 mm to (-76.5, 51.0), turned to 270 degrees
- moved C2 201.1 mm to (-86.5, -1.00)
- moved D2 200.7 mm to (-54.5, 51.0), turned to 90 degrees
- moved C1 200.7 mm to (-86.5, 5.00)
- moved C3 200.4 mm to (-86.5, -8.00)
- moved R4 191.6 mm to (-67.5, -120.5), turned to 90 degrees
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Connections:
- net !CE! renamed PQ25798_!CE!
- net !INT! renamed PQ25798_!INT!
- net !QON! renamed PQ25798_!QON!
- removed net 5V0: R1.2, R2.2, R3.2, R4.2
- removed net B5: USB-C1.B5
- removed net D+: IC5.6_D+, USB-C1.A6, USB-C1.B6
- removed net D-: IC5.7_D-, USB-C1.A7, USB-C1.B7
- removed net SCL: IC5.14_SCL, R4.1
- removed net SDA: IC5.15_SDA, R2.1
- removed net STAT: IC5.1, IC5.1_STAT, R3.1
- new net 3V3: R1.2, R2.2, R4.2, R5.2
- new net I2C_SCL: IC5.14_SCL, R2.1
- new net I2C_SDA: IC5.15_SDA, R5.1
- new net PQ25798_STAT: IC5.1, IC5.1_STAT, R4.1
- new net USB_D+: IC5.6_D+
- new net USB_D-: IC5.7_D-
- net BATTERY_MID: now also BATT1.-, BATT2.+; no longer G1.-, G2.+
- net BATTERY_PLUS: now also BATT1.+; no longer G1.+
- net GND: now also BATT2.-, R3.1; no longer G2.-, R5.1, USB-C1.A1, USB-C1.A12, USB-C1.B1, USB-C1.B12, USB-C1.S1, USB-C1.S2, USB-C1.S3, USB-C1.S4
- net PROG: now also R3.2; no longer R5.2
- net V_USB: no longer USB-C1.A4, USB-C1.A9, USB-C1.B4, USB-C1.B9
