File: eagle design/cos/BQ25798.brd (EAGLE design)
At the start: 68 parts, among them IC1 CSD17581Q3A, IC2 CSD17581Q3A, IC3 CSD17581Q3A, IC4 CSD17581Q3A, IC5 LMR34206SC3QRNXRQ1, IC6 PQ25798RQMT, IC7 CSD17581Q3A

Commit message: - added STM32 Nucleo board layout (NUCLEO-F072RB) for future USB C testing & microcontroller support
Parts:
- added J5, J6: 61300211121, Headers:61300211121
- added NUCLEO1: (no value), ST_NUCLEO-F410RB:NUCLEO
- C11: value 47n/50V -> 0.1u/50V; device rcl:C0805 -> rcl:C0402
- C6: value 4.7n/50V -> 10u/50V; device rcl:C0805 -> rcl:C1206
- C7: value 10u/50V -> 4.7n/50V; device rcl:C1206 -> rcl:C0805
- C8: value 0.1u/50V -> 10u/50V; device rcl:C0402 -> rcl:C1206
- C9: value 10u/50V -> 47n/50V; device rcl:C1206 -> rcl:C0805
- R1: value 8.2k,0.1% -> 0.01R,1W,0.5%; device rcl:R0805 -> rcl:R0402
- R10: value 100R -> 5.24k; device rcl:R0805 -> rcl:R0402
- R11: value 103AT-2 10k NTC -> 33.01k
- R12: value 10k -> 100R; device rcl:R0402 -> rcl:R0805
- R13: value 0.01R,1W,0.5% -> 103AT-2 10k NTC
- R14: value 0.01R,1W,0.5% -> 10k
- R2: value 10k -> 0.01R,1W,0.5%
- R3: value 10k -> 8.2k,0.1%; device rcl:R0402 -> rcl:R0805
- R6: value 100k -> 10k
- R7: value 127k -> 10k
- R8: value 5.24k -> 100k
- R9: value 33.01k -> 127k
- moved R1 319.7 mm to (-271.8, -167.6)
- moved R13 318.3 mm to (-137.5, 121.0), turned to 270 degrees
- moved C6 274.8 mm to (-256.0, 145.5), turned to 0 degrees
- moved C7 274.8 mm to (-142.0, -104.5), turned to 270 degrees
- moved C8 269.3 mm to (-256.0, 138.5), turned to 0 degrees
- moved R12 232.3 mm to (-182.5, 97.0)
- moved R2 206.1 mm to (-271.8, -177.8), turned to 0 degrees
- moved C11 192.3 mm to (-140.0, -104.5), turned to 270 degrees
- moved R14 148.8 mm to (-131.0, -129.5)
- moved R6 136.2 mm to (-219.0, 23.5), turned to 90 degrees
- moved R7 129.7 mm to (-215.0, 23.5), turned to 90 degrees
- moved R3 123.2 mm to (-205.0, 145.0), turned to 0 degrees
- moved C9 74.5 mm to (-237.0, 66.5)
- moved R10 49.0 mm to (-143.0, 126.0), turned to 270 degrees
- moved R4 22.1 mm to (-241.0, 26.0)
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Connections:
- removed net N$8: R16.2, TP8.TP
- new net VOUT: J6.1, R16.2, TP8.TP
- net !PG!: now also R14.2; no longer R12.2
- net 3V3: now also R14.1, R6.2, R7.2; no longer R12.1, R2.2, R3.2
- net BATP: now also R12.1; no longer R10.1
- net BAT_PP: now also R12.2; no longer R10.2
- net BTST1: now also C9.1; no longer C10.1
- net BTST2: now also C10.2; no longer C11.2
- net GND: now also C11.2, J5.2, J6.2, NUCLEO1.AGND, NUCLEO1.GND, NUCLEO1.GND1_1, NUCLEO1.GND1_2, NUCLEO1.GND3, NUCLEO1.GND4_1, NUCLEO1.GND4_2, NUCLEO1.GND5_1, NUCLEO1.GND5_2, NUCLEO1.GND6, R13.2, R3.1, R8.1; no longer C9.2, R1.1, R6.1, R9.2
- net I2C_SCL: now also R6.1; no longer R4.1
- net I2C_SDA: now also R7.1; no longer R5.1
- net ILIM_HIZ: now also R8.2, R9.1; no longer R6.2, R7.1
- net PQ25798_!INT!: now also R4.1; no longer R2.1
- net PQ25798_STAT: now also R5.1; no longer R3.1
- net PROG: now also R3.2; no longer R1.2
- net REGN: now also R10.1, R9.2; no longer R7.2, R8.1
- net SOLAR: now also J5.1, R1.1; no longer R13.1
- net SW1: now also C9.2; no longer C10.2
- net SW2: now also C10.1; no longer C11.1
- net TS: now also R10.2, R13.1; no longer R8.2, R9.1
- net VAC1: now also R2.2; no longer R14.2
- net VAC2: now also R1.2; no longer R13.2
- net VBUS: now also C6.1, C8.1; no longer C7.1, C9.1
- net VIN: now also C11.1, C7.1; no longer C6.1, C8.1
- net V_USB: now also R2.1; no longer R14.1
Other:
- board outline added: 70 x 82.5 mm
