File: eagle design/cos/Čos v0.1.sch (EAGLE design)
At the start: 3 parts, among them X101 22-23-2021, X102 22-23-2021

Commit message: specified input&output capacitors, zener voltage
Other:
- note added: "EMVA101ADA220MHA0G"
- note added: "EMZS350ARA471MHA0G"
- note added: "Vzener: approx. <=20V"
Changed lines of the file:
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@@
 <sheet>
 <plain>
+<text x="40.64" y="83.82" size="1.778" layer="96" rot="R180">Vzener: approx. &lt;=20V</text>
 </plain>
 <instances>
@@
 <sheet>
 <plain>
+<text x="63.5" y="68.58" size="1.778" layer="96" rot="R270">EMZS350ARA471MHA0G</text>
+<text x="109.22" y="66.04" size="1.778" layer="96" rot="R270">EMVA101ADA220MHA0G</text>
 </plain>
 <instances>
