File: eagle design/mj818/MJ818 clone - all driver - prod.sch (EAGLE design)
At the start: 41 parts, among them IC1 MAX16839, IC2 ATTINY4313-MMH, IC3 PBRC8.00GR50X000, IC4 MCP2515, IC5 LDK320M50R, IC6 MCP2561-2, IC7 MAX16820, IC8 SQA470EEJ-T1_GE3

Commit message: - 1st version with larger TH wire connectors
Parts:
- BAT+, GND: device signal testpoint:TPTH-0.9MM -> signal testpoint:TPTH-1.2MM
- H, L: device signal testpoint:TPSMT-1.2MM -> signal testpoint:TPTH-1.2MM
