File: eagle design/mj818/MJ818 clone - rev.5 - SN Mini2 - TCAN334 - prod.brd (EAGLE design)
At the start: 35.5 x 35.5 mm, 40 parts, among them IC202 LDK320AM33R, IC302 STM32F042G6U6, IC401 TCAN334, IC506 MAX16820, IC507 SQA470EEJ-T1_GE3, IC601 MAX16839

Commit message: - generated gerbers - sent board to the FAB
Other:
- board text added: "MJ818 clone SuperNova Mini2 ejovrh rev. 5a"
- board text removed: "Mj818 clone SuperNova Mini2 ejovrh rev. 5a"
Changed lines of the file:
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@@
 <grid distance="0.25" unitdist="mm" unit="mm" style="lines" multiple="1" display="yes" altdistance="0.125" altunitdist="mm" altunit="mm"/>
 <layers>
-<layer number="1" name="Top" color="4" fill="1" visible="yes" active="yes"/>
+<layer number="1" name="Top" color="4" fill="1" visible="no" active="yes"/>
 <layer number="2" name="Route2" color="1" fill="3" visible="no" active="yes"/>
 <layer number="3" name="Route3" color="17" fill="1" visible="no" active="no"/>
@@
 <layer number="14" name="Route14" color="22" fill="1" visible="no" active="no"/>
 <layer number="15" name="Route15" color="4" fill="6" visible="no" active="yes"/>
-<layer number="16" name="Bottom" color="1" fill="1" visible="no" active="yes"/>
+<layer number="16" name="Bottom" color="1" fill="1" visible="yes" active="yes"/>
 <layer number="17" name="Pads" color="2" fill="1" visible="yes" active="yes"/>
 <layer number="18" name="Vias" color="2" fill="1" visible="yes" active="yes"/>
 <layer number="19" name="Unrouted" color="6" fill="1" visible="yes" active="yes"/>
 <layer number="20" name="Dimension" color="24" fill="1" visible="yes" active="yes"/>
-<layer number="21" name="tPlace" color="7" fill="1" visible="yes" active="yes"/>
-<layer number="22" name="bPlace" color="7" fill="1" visible="no" active="yes"/>
-<layer number="23" name="tOrigins" color="15" fill="1" visible="yes" active="yes"/>
-<layer number="24" name="bOrigins" color="15" fill="1" visible="no" active="yes"/>
-<layer number="25" name="tNames" color="7" fill="1" visible="yes" active="yes"/>
-<layer number="26" name="bNames" color="7" fill="1" visible="no" active="yes"/>
+<layer number="21" name="tPlace" color="7" fill="1" visible="no" active="yes"/>
+<layer number="22" name="bPlace" color="7" fill="1" visible="yes" active="yes"/>
+<layer number="23" name="tOrigins" color="15" fill="1" visible="no" active="yes"/>
+<layer number="24" name="bOrigins" color="15" fill="1" visible="yes" active="yes"/>
+<layer number="25" name="tNames" color="7" fill="1" visible="no" active="yes"/>
+<layer number="26" name="bNames" color="7" fill="1" visible="yes" active="yes"/>
 <layer number="27" name="tValues" color="7" fill="1" visible="no" active="yes"/>
 <layer number="28" name="bValues" color="7" fill="1" visible="no" active="yes"/>
-<layer number="29" name="tStop" color="7" fill="3" visible="yes" active="yes"/>
-<layer number="30" name="bStop" color="7" fill="6" visible="no" active="yes"/>
+<layer number="29" name="tStop" color="7" fill="3" visible="no" active="yes"/>
+<layer number="30" name="bStop" color="7" fill="6" visible="yes" active="yes"/>
 <layer number="31" name="tCream" color="7" fill="4" visible="no" active="yes"/>
 <layer number="32" name="bCream" color="7" fill="5" visible="no" active="yes"/>
@@
 <layer number="37" name="tTest" color="7" fill="1" visible="no" active="yes"/>
 <layer number="38" name="bTest" color="7" fill="1" visible="no" active="yes"/>
-<layer number="39" name="tKeepout" color="4" fill="11" visible="yes" active="yes"/>
-<layer number="40" name="bKeepout" color="1" fill="11" visible="no" active="yes"/>
-<layer number="41" name="tRestrict" color="4" fill="10" visible="yes" active="yes"/>
-<layer number="42" name="bRestrict" color="1" fill="10" visible="no" active="yes"/>
+<layer number="39" name="tKeepout" color="4" fill="11" visible="no" active="yes"/>
+<layer number="40" name="bKeepout" color="1" fill="11" visible="yes" active="yes"/>
+<layer number="41" name="tRestrict" color="4" fill="10" visible="no" active="yes"/>
+<layer number="42" name="bRestrict" color="1" fill="10" visible="yes" active="yes"/>
 <layer number="43" name="vRestrict" color="2" fill="10" visible="yes" active="yes"/>
 <layer number="44" name="Drills" color="7" fill="1" visible="no" active="yes"/>
@@
 <layer number="49" name="Reference" color="7" fill="1" visible="no" active="yes"/>
 <layer number="50" name="dxf" color="7" fill="1" visible="no" active="no"/>
-<layer number="51" name="tDocu" color="7" fill="1" visible="yes" active="yes"/>
-<layer number="52" name="bDocu" color="7" fill="1" visible="no" active="yes"/>
+<layer number="51" name="tDocu" color="7" fill="1" visible="no" active="yes"/>
+<layer number="52" name="bDocu" color="7" fill="1" visible="yes" active="yes"/>
 <layer number="53" name="tGND_GNDA" color="7" fill="9" visible="no" active="no"/>
 <layer number="54" name="bGND_GNDA" color="1" fill="9" visible="no" active="no"/>
@@
 <dimension x1="-14" y1="0" x2="14" y2="0" x3="0" y3="-23" textsize="1.778" layer="47" dtype="horizontal"/>
 <dimension x1="-16" y1="-1" x2="16" y2="-1" x3="0" y3="-29" textsize="1.778" layer="47" dtype="horizontal"/>
-<text x="0" y="4.5" size="1" layer="29" font="vector" ratio="15" rot="R180" align="center">Mj818 clone
+<text x="0" y="4.5" size="1" layer="29" font="vector" ratio="15" rot="R180" align="center">MJ818 clone
 SuperNova Mini2
 ejovrh rev. 5a</text>
@@
 <text x="-0.25" y="7.5" size="0.75" layer="22" font="vector" rot="MR0" align="center">BAT+</text>
 <text x="7.5" y="7.5" size="1" layer="22" font="vector" rot="MR180" align="center">GND</text>
+<wire x1="5" y1="8.25" x2="9" y2="8.25" width="0.1524" layer="22"/>
+<wire x1="9" y1="8.25" x2="9" y2="6.75" width="0.1524" layer="22"/>
+<wire x1="9" y1="6.75" x2="5" y2="6.75" width="0.1524" layer="22"/>
+<wire x1="-1.75" y1="8.25" x2="2.25" y2="8.25" width="0.1524" layer="22"/>
+<wire x1="-1.75" y1="8.25" x2="-1.75" y2="6.75" width="0.1524" layer="22"/>
+<wire x1="-1.75" y1="6.75" x2="2.25" y2="6.75" width="0.1524" layer="22"/>
 </plain>
 <attributes>
