File: eagle design/mj818/MJ818 clone - rev.5 - SN Mini2 - TCAN334 - prod.sch (EAGLE design)
At the start: 9 parts

Commit message: - renamed prod brd & sch files to reflect development for the SuperNova Mini2 housing - added docu & info to reflect housing design
Parts:
- removed R101, R102: 10k, rcl:R-EU_R0402
Connections:
- removed net DIM_BRAKE: R101.2
- removed net DIM_REAR: R102.2
- net GND: no longer R101.1, R102.1
Other:
- note added: "SuperNova Mini2 housing"
- note removed: "???"

Commit message: - rough routing complete - corrected STM32 pin assignment of prod to match POC - ERC & DRC check out
Parts:
- removed TP103: LED anode, signal testpoint:TP
- removed TP104: LED cathode, signal testpoint:TP
- renumbered SWD101 to SWD1
Connections:
- removed net LED_AN: TP103.TP$1
- removed net LED_CA: TP104.TP$1
Other:
- note added: "SuperNova Mini2 housing HW rev.5a"
- note added: "timer2 channel1 PWM"
- note added: "timer3 channel1 PWM"
- note removed: "I2C1 SCL"
- note removed: "I2C1 SDA"
- note removed: "SPI1 MISO"
- note removed: "SPI1 MOSI"
- note removed: "SuperNova Mini2 housing"
- note removed: "USART1 rx"
- note removed: "USART1 tx"
- note removed: "external interrupt 0"
- note removed: "external interrupt 1"
- note removed: "red LED Cree XPERED-L1-R250-00401"
- note removed: "timer2 channel1"
- note removed: "timer3 channel 2"
- note removed: "timer3 channel4"

Commit message: - changed size of shunt for rear light to 1206 - finished routing - created BOM - ERC & DRC check out ok
Other:
- note added: "2"
- note added: "3"
- note added: "4"
- note added: "5"
- note added: "6"

Commit message: - generated gerbers - sent board to the FAB
Parts:
- added CONN1: HR30-6R-6P(71), HR30-6R-6P - PushPull Receptacle:HR-30-6R-6X
Connections:
- net BAT+: now also CONN1.2
- net CAN_H: now also CONN1.1
- net CAN_L: now also CONN1.6
- net GND: now also CONN1.5
