File: eagle design/mj818/MJ818 rev.5b - SN Mini2.sch (EAGLE design)
At the start: 8 parts

Commit message: /// start of MJ818 rev.5b - SN Mini2 /// - added CAN protection diode - added power supervisor - replaced CAN solder bridges with 0402 resistors - adapted silkscreen stuff a bit - deleted old original mj818 MagicShine board/schematic - renamed files, updated HW rev. in sch & brd
Parts:
- removed TP1: CAN high, signal testpoint:TPTH-0.9
- removed TP2: CAN low, signal testpoint:TPTH-0.9
Connections:
- net CAN_H: no longer TP1.TP$1
- net CAN_L: no longer TP2.TP$1
Other:
- note added: "0V"
- note added: "7"
- note added: "<5.8V"
- note added: "Dout"
- note added: "I2C: 0x44"
- note added: "MJ818 SuperNova Mini2 HW rev.5b"
- note removed: "SuperNova Mini2 housing HW rev.5a"
