File: eagle design/mj808/MJ808 clone - rev.5 - TCAN334 - poc.sch (EAGLE design)
At the start: 7 parts, among them J1 CAN, J2 Power Supply, J3 LED

Commit message: board revision 5a: - removed CAN infra shutdown pin, since it is not needed
Changed lines of the file:
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@@
 <port name="RED_LED" side="right" coord="-2.54" direction="hiz"/>
 <port name="DIM_FRONT" side="top" coord="12.7" direction="out"/>
-<port name="!SHDN!" side="bottom" coord="-15.24" direction="out"/>
 </ports>
 <variantdefs>
@@
 <text x="137.16" y="142.24" size="1.778" layer="98">GPIO</text>
 <text x="137.16" y="139.7" size="1.778" layer="98">GPIO</text>
-<text x="162.56" y="137.16" size="1.778" layer="98">GPIO</text>
+<text x="137.16" y="137.16" size="1.778" layer="98">GPIO</text>
 <text x="160.02" y="119.38" size="1.778" layer="98">GPIO</text>
 </plain>
@@
 <wire x1="129.54" y1="91.44" x2="149.86" y2="91.44" width="0.1524" layer="91"/>
 <pinref part="IC2" gate="G$1" pin="EVENTOUT,TSC_G5_IO1,TIM2_CH2,SPI1_SCK,I2S1_CK-PB3_24"/>
-</segment>
-</net>
-<net name="!SHDN!" class="0">
-<segment>
-<wire x1="129.54" y1="137.16" x2="152.4" y2="137.16" width="0.1524" layer="91"/>
-<label x="152.4" y="137.16" size="1.778" layer="95" xref="yes"/>
-<pinref part="IC2" gate="G$1" pin="ADC_IN4,USB_NOE,USART2_CK,TSC_G2_IO1,TIM14_CH1,SPI1_NSS,I2S1_WS-PA4_10"/>
 </segment>
 </net>
@@
 <port name="RXCAN" side="left" coord="2.54" direction="out"/>
 <port name="!STBY!" side="left" coord="0" direction="in"/>
-<port name="!SHDN!" side="left" coord="-2.54" direction="in"/>
 </ports>
 <variantdefs>
@@
 <sheet>
 <plain>
-<text x="40.64" y="71.12" size="1.778" layer="97" rot="R180">internal pulldown</text>
+<text x="66.04" y="71.12" size="1.778" layer="97" rot="R180" align="top-left">internal pulldown</text>
 <text x="40.64" y="68.58" size="1.778" layer="97" rot="R180">internal pulldown</text>
 </plain>
@@
 <wire x1="142.24" y1="104.14" x2="142.24" y2="101.6" width="0.1524" layer="91"/>
 <label x="142.24" y="101.6" size="0.8128" layer="95"/>
-</segment>
-</net>
-<net name="!SHDN!" class="0">
-<segment>
-<pinref part="IC1" gate="G$1" pin="5_SHDN"/>
-<wire x1="68.58" y1="71.12" x2="50.8" y2="71.12" width="0.1524" layer="91"/>
-<label x="50.8" y="71.12" size="1.778" layer="95" rot="R180" xref="yes"/>
 </segment>
 </net>
@@
 </segment>
 </net>
-<net name="!SHDN!" class="0">
-<segment>
-<portref moduleinst="CAN_INFRA" port="!SHDN!"/>
-<wire x1="149.86" y1="78.74" x2="142.24" y2="78.74" width="0.1524" layer="91"/>
-<portref moduleinst="STM32F04" port="!SHDN!"/>
-<wire x1="142.24" y1="101.6" x2="142.24" y2="78.74" width="0.1524" layer="91"/>
-</segment>
-</net>

Commit message: - updated mj8x8 template board and schematic with previous changes - added TODOs for mj808/818/828 boards (rerouting, mostly)
Other:
- note added: "TODO: - move PB3 (tim2 ch2) to PAx - move PB1 (gpio) to PAx - move PB0 (exti0) to PA0 - move PB4/5 (gpio) tp PAx"
Changed lines of the file:
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@@
 <text x="15.24" y="205.74" size="6.4516" layer="98" rot="R180" align="bottom-right">MJ8x8 - generic</text>
 <text x="180.34" y="165.1" size="6.4516" layer="94">???</text>
+<text x="271.78" y="63.5" size="1.778" layer="91">TODO:
+- move PB3 (tim2 ch2) to PAx
+- move PB1 (gpio) to PAx
+- move PB0 (exti0) to PA0
+- move PB4/5 (gpio) tp PAx</text>
 </plain>
 <moduleinsts>

Commit message: board revision 5a: - removed CAN infra shutdown pin, since it is not needed
Other:
- note removed: "TODO: - move PB3 (tim2 ch2) to PAx - move PB1 (gpio) to PAx - move PB0 (exti0) to PA0 - move PB4/5 (gpio) tp PAx"
Changed lines of the file:
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@@
 <parts>
 <part name="SUPPLY1" library="Power_Symbols" library_urn="urn:adsk.eagle:library:16502351" deviceset="GND-BAR" device="" value="GND"/>
-<part name="R5" library="rcl" library_urn="urn:adsk.eagle:library:334" deviceset="R-EU_" device="R0805" package3d_urn="urn:adsk.eagle:package:23553/2" value="60"/>
+<part name="R5" library="rcl" library_urn="urn:adsk.eagle:library:334" deviceset="R-EU_" device="R0805" package3d_urn="urn:adsk.eagle:package:23553/2" value="120"/>
 <part name="C5" library="rcl" library_urn="urn:adsk.eagle:library:334" deviceset="C-EU" device="C0402" package3d_urn="urn:adsk.eagle:package:23626/2" value="0.1μF"/>
 <part name="SUPPLY2" library="Power_Symbols" library_urn="urn:adsk.eagle:library:16502351" deviceset="GND-BAR" device="" value="GND"/>
 <part name="SUPPLY3" library="Power_Symbols" library_urn="urn:adsk.eagle:library:16502351" deviceset="GND-BAR" device="" value="GND"/>
 <part name="CAN_INFRA" library="frames" library_urn="urn:adsk.eagle:library:229" deviceset="DINA5_L" device="" value="CAN_INFRA"/>
+<part name="SJ1" library="rcl" library_urn="urn:adsk.eagle:library:334" deviceset="R-EU_" device="R0402" package3d_urn="urn:adsk.eagle:package:23547/3" value="CAN termination"/>
 <part name="IC1" library="TCAN33x - 3.3V CAN Transciever" deviceset="CAN33X" device="" value="TCAN334"/>
-<part name="R1" library="rcl" library_urn="urn:adsk.eagle:library:334" deviceset="R-EU_" device="R0805" package3d_urn="urn:adsk.eagle:package:23553/2" value="60"/>
-<part name="C1" library="rcl" library_urn="urn:adsk.eagle:library:334" deviceset="C-EU" device="C0402" package3d_urn="urn:adsk.eagle:package:23626/2" value="47nF"/>
-<part name="SUPPLY4" library="Power_Symbols" library_urn="urn:adsk.eagle:library:16502351" deviceset="GND-BAR" device="" value="GND"/>
+<part name="TP1" library="testpad" library_urn="urn:adsk.eagle:library:385" deviceset="PTR1" device="PAD1-13" package3d_urn="urn:adsk.eagle:package:27946/1"/>
+<part name="TP2" library="testpad" library_urn="urn:adsk.eagle:library:385" deviceset="PTR1" device="PAD1-13" package3d_urn="urn:adsk.eagle:package:27946/1"/>
 </parts>
 <sheets>
@@
 <attribute name="SHEET" x="154.305" y="5.08" size="2.54" layer="94"/>
 </instance>
+<instance part="SJ1" gate="G$1" x="142.24" y="109.22" smashed="yes" rot="R90">
+<attribute name="NAME" x="139.7" y="109.22" size="1.778" layer="95" rot="R180"/>
+<attribute name="VALUE" x="144.78" y="109.22" size="1.778" layer="96"/>
+</instance>
 <instance part="IC1" gate="G$1" x="83.82" y="73.66" smashed="yes">
 <attribute name="NAME" x="76.2" y="83.82" size="1.27" layer="95" font="vector" align="center"/>
 <attribute name="VALUE" x="76.2" y="55.88" size="1.27" layer="95" font="vector" align="center"/>
 </instance>
-<instance part="R1" gate="G$1" x="142.24" y="109.22" smashed="yes" rot="R90">
-<attribute name="NAME" x="144.78" y="111.76" size="1.778" layer="95"/>
-<attribute name="VALUE" x="144.78" y="109.22" size="1.778" layer="96"/>
-</instance>
-<instance part="C1" gate="G$1" x="154.94" y="99.06" smashed="yes">
-<attribute name="NAME" x="157.48" y="99.06" size="1.778" layer="95"/>
-<attribute name="VALUE" x="157.48" y="96.52" size="1.778" layer="96"/>
-</instance>
-<instance part="SUPPLY4" gate="G$1" x="154.94" y="88.9" smashed="yes">
-<attribute name="VALUE" x="154.94" y="86.995" size="1.778" layer="96" align="center"/>
+<instance part="TP1" gate="G$1" x="119.38" y="81.28" smashed="yes" rot="R180">
+<attribute name="NAME" x="121.92" y="81.28" size="1.778" layer="95"/>
+<attribute name="TP_SIGNAL_NAME" x="118.11" y="83.82" size="1.778" layer="97" rot="R180"/>
+</instance>
+<instance part="TP2" gate="G$1" x="119.38" y="71.12" smashed="yes">
+<attribute name="NAME" x="121.92" y="71.12" size="1.778" layer="95"/>
+<attribute name="TP_SIGNAL_NAME" x="120.65" y="68.58" size="1.778" layer="97"/>
 </instance>
 </instances>
@@
 <pinref part="IC1" gate="G$1" pin="2_GND"/>
 </segment>
-<segment>
-<pinref part="C1" gate="G$1" pin="2"/>
-<pinref part="SUPPLY4" gate="G$1" pin="GND"/>
-<wire x1="154.94" y1="91.44" x2="154.94" y2="93.98" width="0.1524" layer="91"/>
-</segment>
 </net>
 <net name="CAN_H" class="0">
@@
 <wire x1="119.38" y1="78.74" x2="127" y2="78.74" width="0.1524" layer="91"/>
 <label x="127" y="78.74" size="1.778" layer="95" xref="yes"/>
+<pinref part="TP1" gate="G$1" pin="TP"/>
+<junction x="119.38" y="78.74"/>
 </segment>
 <segment>
@@
 <segment>
 <wire x1="142.24" y1="114.3" x2="142.24" y2="118.11" width="0.1524" layer="91"/>
+<pinref part="SJ1" gate="G$1" pin="2"/>
 <label x="142.24" y="118.11" size="1.778" layer="95"/>
-<pinref part="R1" gate="G$1" pin="2"/>
 </segment>
 </net>
@@
 <wire x1="119.38" y1="73.66" x2="127" y2="73.66" width="0.1524" layer="91"/>
 <label x="127" y="73.66" size="1.778" layer="95" xref="yes"/>
+<pinref part="TP2" gate="G$1" pin="TP"/>
+<junction x="119.38" y="73.66"/>
 </segment>
 <segment>
@@
 </segment>
 </net>
-<net name="SPLIT" class="3">
+<net name="CAN_JMPR" class="3">
 <segment>
 <pinref part="R5" gate="G$1" pin="2"/>
+<pinref part="SJ1" gate="G$1" pin="1"/>
 <wire x1="142.24" y1="104.14" x2="142.24" y2="101.6" width="0.1524" layer="91"/>
 <label x="142.24" y="101.6" size="0.8128" layer="95"/>
-<pinref part="R1" gate="G$1" pin="1"/>
-<pinref part="C1" gate="G$1" pin="1"/>
-<wire x1="154.94" y1="101.6" x2="142.24" y2="101.6" width="0.1524" layer="91"/>
-<junction x="142.24" y="101.6"/>
 </segment>
 </net>
@@
 <text x="15.24" y="205.74" size="6.4516" layer="98" rot="R180" align="bottom-right">MJ8x8 - generic</text>
 <text x="180.34" y="165.1" size="6.4516" layer="94">???</text>
-<text x="271.78" y="63.5" size="1.778" layer="91">TODO:
-- move PB3 (tim2 ch2) to PAx
-- move PB1 (gpio) to PAx
-- move PB0 (exti0) to PA0
-- move PB4/5 (gpio) tp PAx</text>
 </plain>
 <moduleinsts>
