File: eagle design/mj808/MJ808 clone - rev.5 - TCAN334 - SN E3 - prod.brd (EAGLE design)
At the start: 36.5 x 36.5 mm, 37 parts, among them IC202 LDK320AM33R, IC302 STM32F042G6U6, IC401 TCAN334, IC506 MAX16820, IC507 SQA470EEJ-T1_GE3, IC602 MAX6816EUS+T

Commit message: MJ818 SuperNova Mini2: - added position key into PCB and spacers; updated gerber, dwg and stl
mj513 - grip:
- corrected bushing dimensions

in mj8x8-foo:
- minor corrections

general board-wide effort:
- replaced pinhead with 0.9mm TH
- added 2nd CAN H & L solder contact
- unified sch nets and drawings

in mj8x8 foo:
- developed rev.1b mj-foo device with voltage detector and CAN TVS protection

in mj808 design:
- updated front led shunt resistor to 0.18 Ohm

in mj8x8:
- added HR30-6R-6P - PushPull Receptacle.lbr receptable
Parts:
- R504: value WSLT2010R2200FEB18 / 0.22Ohm 1W -> 0.18R
Changed lines of the file:
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@@
 <grid distance="0.25" unitdist="mm" unit="mm" style="lines" multiple="1" display="yes" altdistance="0.125" altunitdist="mm" altunit="mm"/>
 <layers>
-<layer number="1" name="Top" color="4" fill="1" visible="no" active="yes"/>
-<layer number="2" name="Route2" color="1" fill="3" visible="yes" active="yes"/>
+<layer number="1" name="Top" color="4" fill="1" visible="yes" active="yes"/>
+<layer number="2" name="Route2" color="1" fill="3" visible="no" active="yes"/>
 <layer number="3" name="Route3" color="4" fill="3" visible="no" active="no"/>
 <layer number="4" name="Route4" color="1" fill="4" visible="no" active="no"/>
@@
 <layer number="19" name="Unrouted" color="6" fill="1" visible="yes" active="yes"/>
 <layer number="20" name="Dimension" color="24" fill="1" visible="yes" active="yes"/>
-<layer number="21" name="tPlace" color="7" fill="1" visible="no" active="yes"/>
+<layer number="21" name="tPlace" color="7" fill="1" visible="yes" active="yes"/>
 <layer number="22" name="bPlace" color="7" fill="1" visible="no" active="yes"/>
-<layer number="23" name="tOrigins" color="15" fill="1" visible="no" active="yes"/>
+<layer number="23" name="tOrigins" color="15" fill="1" visible="yes" active="yes"/>
 <layer number="24" name="bOrigins" color="15" fill="1" visible="no" active="yes"/>
-<layer number="25" name="tNames" color="7" fill="1" visible="no" active="yes"/>
+<layer number="25" name="tNames" color="7" fill="1" visible="yes" active="yes"/>
 <layer number="26" name="bNames" color="7" fill="1" visible="no" active="yes"/>
 <layer number="27" name="tValues" color="7" fill="1" visible="no" active="yes"/>
 <layer number="28" name="bValues" color="7" fill="1" visible="no" active="yes"/>
-<layer number="29" name="tStop" color="7" fill="3" visible="no" active="yes"/>
+<layer number="29" name="tStop" color="7" fill="3" visible="yes" active="yes"/>
 <layer number="30" name="bStop" color="7" fill="6" visible="no" active="yes"/>
 <layer number="31" name="tCream" color="7" fill="4" visible="no" active="yes"/>
@@
 <layer number="37" name="tTest" color="7" fill="1" visible="no" active="yes"/>
 <layer number="38" name="bTest" color="7" fill="1" visible="no" active="yes"/>
-<layer number="39" name="tKeepout" color="4" fill="11" visible="no" active="yes"/>
+<layer number="39" name="tKeepout" color="4" fill="11" visible="yes" active="yes"/>
 <layer number="40" name="bKeepout" color="1" fill="11" visible="no" active="yes"/>
-<layer number="41" name="tRestrict" color="4" fill="10" visible="no" active="yes"/>
+<layer number="41" name="tRestrict" color="4" fill="10" visible="yes" active="yes"/>
 <layer number="42" name="bRestrict" color="1" fill="10" visible="no" active="yes"/>
 <layer number="43" name="vRestrict" color="2" fill="10" visible="yes" active="yes"/>
@@
 <layer number="49" name="Reference" color="7" fill="1" visible="no" active="yes"/>
 <layer number="50" name="dxf" color="7" fill="1" visible="no" active="no"/>
-<layer number="51" name="tDocu" color="7" fill="1" visible="no" active="yes"/>
+<layer number="51" name="tDocu" color="7" fill="1" visible="yes" active="yes"/>
 <layer number="52" name="bDocu" color="7" fill="1" visible="no" active="yes"/>
 <layer number="53" name="tGND_GNDA" color="7" fill="9" visible="no" active="no"/>
@@
 <attribute name="VALUE" x="12.115" y="0.587" size="1.27" layer="27"/>
 </element>
-<element name="R504" library="rcl" library_urn="urn:adsk.eagle:library:334" package="R2010" package3d_urn="urn:adsk.eagle:package:23551/2" value="WSLT2010R2200FEB18 / 0.22Ohm 1W" x="-5.004" y="-7.75" smashed="yes" rot="R90">
+<element name="R504" library="rcl" library_urn="urn:adsk.eagle:library:334" package="R2010" package3d_urn="urn:adsk.eagle:package:23551/2" value="0.18R" x="-5.004" y="-7.75" smashed="yes" rot="R90">
 <attribute name="NAME" x="-7" y="-7.75" size="0.5" layer="25" font="vector" rot="R270" align="center"/>
 <attribute name="POPULARITY" value="3" x="-5.004" y="-7.75" size="1.778" layer="27" rot="R90" display="off"/>
@@
 <wire x1="8.31" y1="2.94" x2="8.31" y2="1.19" width="0.25" layer="1"/>
 </signal>
-<signal name="SWITCH">
+<signal name="SWITCH" class="3">
 <contactref element="IC602" pad="3_OUT"/>
 <contactref element="IC302" pad="6_PA0"/>
@@
 <via x="-12.25" y="-1.512" extent="1-16" drill="0.35"/>
 </signal>
-<signal name="GREEN">
+<signal name="GREEN" class="4">
 <contactref element="IC302" pad="10_PA4"/>
 <contactref element="LED703" pad="CAT"/>
@@
 <wire x1="3.98" y1="4.5" x2="-1" y2="4.5" width="0.25" layer="15"/>
 </signal>
-<signal name="RED">
+<signal name="RED" class="4">
 <contactref element="IC302" pad="8_PA2"/>
 <contactref element="LED702" pad="CAT"/>
