File: eagle design/mj808/MJ808 rev.5b - SN E3.sch (EAGLE design)
At the start: 10 parts

Commit message: /// start of MJ808 rev.5b - SN E3 /// - added CAN protection diode - added power supervisor - replaced CAN solder bridges with 0402 resistors - adapted silkscreen stuff a bit - renamed files, updated HW rev. in sch & brd
Other:
- note added: "0V"
- note added: "<5.8V"
- note added: "Dout"
- note added: "I2C: 0x44"
- note added: "MJ808 SuperNova E3 HW rev.5b"
- note removed: "SuperNova E3 housing HW rev.5a"
