File: eagle design/mj828/MJ828 - rev.3 - TCAN334 - poc.sch (EAGLE design)
At the start: 6 parts, among them J1 CAN, J2 Power Supply

Commit message: added ADC code for interrupt-based readout
adc.h/adc_actual.c:
- defined adc_t, __adc_t

mj828_adc.c:
- moved ADC init into this file
- implemented adc_ctor()
- implemented _GetVal(), _ReadChannels

mj828.c/.h:
- implemented above changes

MJ828 - rev.3 - TCAN334 - poc.brd/.sch:
- changed voltage divider high resistor value so that a divided 8.4V is less than 3.3V
Other:
- note added: "ideal calculation of divider: BAT+ -- Vbat+ 8.4V -- 2.27 (4.2 per cell) 6.0V -- 1.622 (3.0 per cell)"
Changed lines of the file:
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@@
 <part name="SUPPLY2" library="Power_Symbols" library_urn="urn:adsk.eagle:library:16502351" deviceset="GND-BAR" device="" value="GND"/>
 <part name="R1" library="rcl" library_urn="urn:adsk.eagle:library:334" deviceset="R-EU_" device="R0402" package3d_urn="urn:adsk.eagle:package:23547/3" value="100k"/>
-<part name="R2" library="rcl" library_urn="urn:adsk.eagle:library:334" deviceset="R-EU_" device="R0402" package3d_urn="urn:adsk.eagle:package:23547/3" value="100k"/>
+<part name="R2" library="rcl" library_urn="urn:adsk.eagle:library:334" deviceset="R-EU_" device="R0402" package3d_urn="urn:adsk.eagle:package:23547/3" value="270k"/>
 <part name="SUPPLY1" library="Power_Symbols" library_urn="urn:adsk.eagle:library:16502351" deviceset="GND-BAR" device="" value="GND"/>
 </parts>
@@
 <plain>
 <text x="88.9" y="20.32" size="1.778" layer="90">Voltage Divider for Battery Measurement</text>
+<text x="101.6" y="53.34" size="1.778" layer="97" align="top-left">ideal calculation of divider:
+BAT+ -- Vbat+
+8.4V -- 2.27 (4.2 per cell)
+6.0V -- 1.622 (3.0 per cell)</text>
 </plain>
 <instances>

Commit message: for mj828 changed Vbat+ voltage divider resistors to 0.1% 300k and 100k adjusted ADC values in _DisplayBatteryVoltage() accordingly
Other:
- note added: "ideal calculation of divider: BAT+ -- Vbat+ 8.4V (4.2 per cell) -- 2.1V 6.0V (3.0 per cell) -- 1.5V"
- note removed: "ideal calculation of divider: BAT+ -- Vbat+ 8.4V -- 2.27 (4.2 per cell) 6.0V -- 1.622 (3.0 per cell)"
Changed lines of the file:
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@@
 <part name="VOLTAGE_DIVIDER" library="frames" library_urn="urn:adsk.eagle:library:229" deviceset="A5L-LOC" device="" value="VOLTAGE_DIVIDER"/>
 <part name="SUPPLY2" library="Power_Symbols" library_urn="urn:adsk.eagle:library:16502351" deviceset="GND-BAR" device="" value="GND"/>
-<part name="R1" library="rcl" library_urn="urn:adsk.eagle:library:334" deviceset="R-EU_" device="R0402" package3d_urn="urn:adsk.eagle:package:23547/3" value="100k"/>
-<part name="R2" library="rcl" library_urn="urn:adsk.eagle:library:334" deviceset="R-EU_" device="R0402" package3d_urn="urn:adsk.eagle:package:23547/3" value="270k"/>
+<part name="R1" library="rcl" library_urn="urn:adsk.eagle:library:334" deviceset="R-EU_" device="R0402" package3d_urn="urn:adsk.eagle:package:23547/3" value="100k 0.1%"/>
+<part name="R2" library="rcl" library_urn="urn:adsk.eagle:library:334" deviceset="R-EU_" device="R0402" package3d_urn="urn:adsk.eagle:package:23547/3" value="300k 0.1%"/>
 <part name="SUPPLY1" library="Power_Symbols" library_urn="urn:adsk.eagle:library:16502351" deviceset="GND-BAR" device="" value="GND"/>
 </parts>
@@
 <text x="101.6" y="53.34" size="1.778" layer="97" align="top-left">ideal calculation of divider:
 BAT+ -- Vbat+
-8.4V -- 2.27 (4.2 per cell)
-6.0V -- 1.622 (3.0 per cell)</text>
+8.4V (4.2 per cell) -- 2.1V
+6.0V (3.0 per cell) -- 1.5V</text>
 </plain>
 <instances>

Commit message: board revision 5a: - removed CAN infra shutdown pin, since it is not needed
Changed lines of the file:
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@@
 <port name="HIGH_IN" side="bottom" coord="22.86" direction="in"/>
 <port name="VBAT+" side="top" coord="12.7" direction="in"/>
-<port name="!SHDN!" side="bottom" coord="-15.24" direction="out"/>
 </ports>
 <variantdefs>
@@
 </segment>
 </net>
-<net name="!SHDN!" class="0">
-<segment>
-<label x="149.86" y="160.02" size="1.778" layer="95" xref="yes"/>
-<pinref part="IC2" gate="G$1" pin="I2C1_SCL,OSC_OUT-PF1_3"/>
-<wire x1="129.54" y1="160.02" x2="149.86" y2="160.02" width="0.1524" layer="91"/>
-</segment>
-</net>
 <net name="CP3" class="3">
 <segment>
@@
 <port name="RXCAN" side="left" coord="2.54" direction="out"/>
 <port name="!STBY!" side="left" coord="0" direction="in"/>
-<port name="!SHDN!" side="left" coord="-2.54" direction="in"/>
 </ports>
 <variantdefs>
@@
 <text x="40.64" y="68.58" size="1.778" layer="97" rot="R180">internal pulldown</text>
 <text x="88.9" y="20.32" size="1.778" layer="90">CAN infrastructure</text>
-<text x="40.64" y="71.12" size="1.778" layer="97" rot="R180">internal pulldown</text>
+<text x="66.04" y="71.12" size="1.778" layer="97" rot="R180" align="top-left">internal pulldown</text>
 </plain>
 <instances>
@@
 <wire x1="142.24" y1="104.14" x2="142.24" y2="101.6" width="0.1524" layer="91"/>
 <label x="142.24" y="101.6" size="0.8128" layer="95"/>
-</segment>
-</net>
-<net name="!SHDN!" class="0">
-<segment>
-<wire x1="50.8" y1="71.12" x2="68.58" y2="71.12" width="0.1524" layer="91"/>
-<label x="50.8" y="71.12" size="1.778" layer="95" rot="R180" xref="yes"/>
-<pinref part="IC1" gate="G$1" pin="5_SHDN"/>
 </segment>
 </net>
@@
 </segment>
 </net>
-<net name="!SHDN!" class="0">
-<segment>
-<portref moduleinst="STM32F04" port="!SHDN!"/>
-<portref moduleinst="CAN_INFRA" port="!SHDN!"/>
-<wire x1="142.24" y1="101.6" x2="142.24" y2="78.74" width="0.1524" layer="91"/>
-<wire x1="142.24" y1="78.74" x2="149.86" y2="78.74" width="0.1524" layer="91"/>
-</segment>
-</net>
