File: eagle design/mj514/MJ514 - rev.1 - POC.sch (EAGLE design)
At the start: 5 parts

Commit message: - added LTC1935 - Boost DC-DC Converter for 12V0 voltage source - added above element to schematic
Parts:
- removed JP1, JP2: (no value), pinhead:PINHD-1X2
- removed JP3: (no value), pinhead:PINHD-1X7
- removed R1, R2: 4k7, rcl:R-EU_R0402
- added JP101: (no value), pinhead:PINHD-1X7
- added JP102, JP103: (no value), pinhead:PINHD-1X2
- added R101, R102: 4k7, rcl:R-EU_R0402
Connections:
- removed net 8V4: JP2.1
- new net BAT+: JP102.1
- net 3V3: now also R101.2, R102.2; no longer R1.2, R2.2
- net GND: now also JP102.2; no longer JP2.2
- net I2C_SCL: now also R101.1; no longer R1.1
- net I2C_SDA: now also R102.1; no longer R2.1
- net MOTOR+: now also JP103.1; no longer JP1.1
- net MOTOR-: now also JP103.2; no longer JP1.2
Other:
- note added: "FB Resistors: VOUT = 1.265V(1 + R1/R2). 12V = 1.265V * (1 + 85.8/10) = 12.09V"
- note added: "Inductor: DS. p. 5: L = 3 (VIN/VOUT) (VOUT – VIN)/(IMAX • f) 8.4V: L= 3 * (8.4/12.0) * (12.0 - 8.4) / (1.5A * 1.2MHz) = 3 * 0.7 / (1.5 * 1.2exp6) = 3 * 3.89exp-7 = 1.17 uH 7.0V: L= 3 * (7/12.0) * (12.0 - 7.0) / (1.5A * 1.2MHz) = 3 * 0.5833 / (1.5 * 1.2exp6) = 3 * 3.24exp-7 = 9.72 uH"

Commit message: mj514 rev.1 PCB first rough layout is complete
Parts:
- removed JP101: (no value), pinhead:PINHD-1X7
- removed JP102, JP103: (no value), pinhead:PINHD-1X2
- removed R101, R102: 4k7, rcl:R-EU_R0402
- added JP3: (no value), pinhead:PINHD-1X2
- added R1, R2: 4k7, rcl:R-EU_R0402
Connections:
- removed net BAT+: JP102.1
- new net 12V: R2.2
- new net FB: R1.2, R2.1
- new net IMODE: R1.2
- new net PMODE: R2.2
- net 3V3: now also R1.2, R2.2; no longer R101.2, R102.2
- net GND: now also R1.1, R2.1; no longer JP102.2
- net I2C_SCL: now also R1.1; no longer R101.1
- net I2C_SDA: now also R2.1; no longer R102.1
- net MOTOR+: now also JP3.1; no longer JP103.1
- net MOTOR-: now also JP3.2; no longer JP103.2
Other:
- note added: "PA0"
- note added: "PA1"
- note added: "PA10"
- note added: "PA11"
- note added: "PA2"
- note added: "PA3"
- note added: "PA4"
- note added: "PA6"
- note added: "PA7"
- note added: "Vmotor_iprop (ADC input): V = R * I = 1k * 1A = 1V"
- note added: "low-pass fcutoff 723.4 Hz"
- note added: "see DS. p. 13"
- note added: "trace endpoints are 1mm vias"

Commit message: moved e14 reverse engineering to seperate branch, moved mj514 POC into POC branch
Parts:
- removed JP3: (no value), pinhead:PINHD-1X2
- removed R1, R2: 4k7, rcl:R-EU_R0402
- added IC1: (no value), AS5601 - Programmable Contactless Encoder:AS5601
- added JP1, JP2: (no value), pinhead:PINHD-1X2
Connections:
- removed net 12V: R2.2
- removed net FB: R1.2, R2.1
- removed net I2C_SCL: R1.1
- removed net I2C_SDA: R2.1
- removed net IMODE: R1.2
- removed net PMODE: R2.2
- new net !STBY!: IC1.8_STB
- new net 8V4: JP2.1
- new net CAN_H: IC1.7_CANH
- new net CAN_L: IC1.6_CANL
- new net RXCAN: IC1.4_RXD
- new net TXCAN: IC1.1_TXD
- net 3V3: now also IC1.3_VCC; no longer R1.2, R2.2
- net GND: now also IC1.2_GND, JP2.2; no longer R1.1, R2.1
- net MOTOR+: now also JP1.1; no longer JP3.1
- net MOTOR-: now also JP1.2; no longer JP3.2
Other:
- note added: "Vdd"
- note added: "VddIO2"
- note added: "Vdda"
- note added: "fixed"
- note added: "internal pulldown"
- note removed: "FB Resistors: VOUT = 1.265V(1 + R1/R2). 12V = 1.265V * (1 + 85.8/10) = 12.09V"
- note removed: "Inductor: DS. p. 5: L = 3 (VIN/VOUT) (VOUT – VIN)/(IMAX • f) 8.4V: L= 3 * (8.4/12.0) * (12.0 - 8.4) / (1.5A * 1.2MHz) = 3 * 0.7 / (1.5 * 1.2exp6) = 3 * 3.89exp-7 = 1.17 uH 7.0V: L= 3 * (7/12.0) * (12.0 - 7.0) / (1.5A * 1.2MHz) = 3 * 0.5833 / (1.5 * 1.2exp6) = 3 * 3.24exp-7 = 9.72 uH"
- note removed: "PA0"
- note removed: "PA1"
- note removed: "PA10"
- note removed: "PA11"
- note removed: "PA2"
- note removed: "PA3"
- note removed: "PA4"
- note removed: "PA6"
- note removed: "PA7"
- note removed: "Vmotor_iprop (ADC input): V = R * I = 1k * 1A = 1V"
- note removed: "low-pass fcutoff 723.4 Hz"
- note removed: "see DS. p. 13"
- note removed: "trace endpoints are 1mm vias"

Commit message: - added AS5601 - Programmable Contactless Encoder and MB85RC - FeRAM, I2C libraries and added them to schematic - defined GPIOs for above ICs
Parts:
- removed IC1: (no value), AS5601 - Programmable Contactless Encoder:AS5601
- added JP3: (no value), pinhead:PINHD-1X7
- added R1, R2: 10k, rcl:R-EU_R0402
Connections:
- removed net !STBY!: IC1.8_STB
- removed net CAN_H: IC1.7_CANH
- removed net CAN_L: IC1.6_CANL
- removed net RXCAN: IC1.4_RXD
- removed net TXCAN: IC1.1_TXD
- new net I2C_SCL: R1.1
- new net I2C_SDA: R2.1
- net 3V3: now also R1.2, R2.2; no longer IC1.3_VCC
- net GND: no longer IC1.2_GND
Other:
- note removed: "Vdd"
- note removed: "VddIO2"
- note removed: "Vdda"
- note removed: "fixed"
- note removed: "internal pulldown"

Commit message: in brd & sch: - corrected/renamed rotary A & B nets - changed Rpullup for I3C bus from 10k to 4k7
Parts:
- R1, R2: value 10k -> 4k7
Changed lines of the file:
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@@
 </segment>
 </net>
-<net name="ROTARY_B" class="0">
+<net name="ROTARY_A" class="0">
 <segment>
 <pinref part="IC1" gate="G$1" pin="A"/>
 <wire x1="78.74" y1="88.9" x2="68.58" y2="88.9" width="0.1524" layer="91"/>
 <label x="68.58" y="88.9" size="1.778" layer="95" rot="R180" xref="yes"/>
-</segment>
-</net>
-<net name="ROTARY_A" class="0">
-<segment>
-<pinref part="IC1" gate="G$1" pin="B"/>
-<wire x1="78.74" y1="86.36" x2="73.66" y2="86.36" width="0.1524" layer="91"/>
-<label x="73.66" y="86.36" size="1.778" layer="95" rot="R180" xref="yes"/>
 </segment>
 </net>
@@
 <wire x1="78.74" y1="81.28" x2="40.64" y2="81.28" width="0.1524" layer="91"/>
 <label x="43.18" y="81.28" size="1.778" layer="95"/>
+</segment>
+</net>
+<net name="ROTARY_B" class="0">
+<segment>
+<pinref part="IC1" gate="G$1" pin="B"/>
+<wire x1="78.74" y1="86.36" x2="73.66" y2="86.36" width="0.1524" layer="91"/>
+<label x="73.66" y="86.36" size="1.778" layer="95" rot="R180" xref="yes"/>
 </segment>
 </net>
@@
 <part name="SUPPLY3" library="Power_Symbols" library_urn="urn:adsk.eagle:library:16502351" deviceset="GND-BAR" device="" value="GND"/>
 <part name="SUPPLY5" library="Power_Symbols" library_urn="urn:adsk.eagle:library:16502351" deviceset="GND-BAR" device="" value="GND"/>
-<part name="R1" library="rcl" library_urn="urn:adsk.eagle:library:334" deviceset="R-EU_" device="R0402" package3d_urn="urn:adsk.eagle:package:23547/3" value="10k"/>
-<part name="R2" library="rcl" library_urn="urn:adsk.eagle:library:334" deviceset="R-EU_" device="R0402" package3d_urn="urn:adsk.eagle:package:23547/3" value="10k"/>
+<part name="R1" library="rcl" library_urn="urn:adsk.eagle:library:334" deviceset="R-EU_" device="R0402" package3d_urn="urn:adsk.eagle:package:23547/3" value="4k7"/>
+<part name="R2" library="rcl" library_urn="urn:adsk.eagle:library:334" deviceset="R-EU_" device="R0402" package3d_urn="urn:adsk.eagle:package:23547/3" value="4k7"/>
 <part name="SUPPLY6" library="Power_Symbols" library_urn="urn:adsk.eagle:library:16502351" deviceset="3V3-CIRCLE" device="" value="3V3"/>
 <part name="SUPPLY7" library="Power_Symbols" library_urn="urn:adsk.eagle:library:16502351" deviceset="3V3-CIRCLE" device="" value="3V3"/>
