File: eagle design/mj514/MJ514 - rev.1 - prod.brd (EAGLE design)
At the start: 49 x 18 mm, 56 parts, among them IC201 LDK320AM33R, IC203 R3119N058A-TR-FE, IC302 STM32F042G6U6, IC401 TCAN334, IC402 SZNUP2105LT1G, IC501 SHT40-AD1F-R2, IC601 MB85RC16PN-G-AMERE1, IC701 AS5601-ASOM, IC801 LT1935ES5#TRMPBF, IC901 DRV8876RGTR

Commit message: in board design: - added current sense resistor calculation - in 12V0 regulator added slow start RC lowpass filter, as per DS. p. 6 - moved 12V_SHDN to PA5
in motor.c/.h:
- code tweaks for angle statistics
- added #if USE_AS5601_PULSE across the code to deactivate not needed code
- in timer16 ISR: added _EndTravelTime and coded setting this variable with the elapsed milliseconds once the travel end is reached
- in timer16 ISR: added code which allows timer16 to continue to run after end travel is reached
- in _StartMotorController() & _StopMotorController() added timer16 interrupt priority change (suspect was some race condition or priority collision)
- set & unset FlagShiftingDone, for above checks
- added #define USE_RAMPUP so that rampup code can be disabled
- cleaned up code by adding #if CURRENT_STATS and #if ANGLE_STATS
- added typecast to get rid of compiler warnings
- added misc. code for testing stuff
- added arrays _PulseCorrection[] and _RawAngleCorrection; these hold corrections which need to be applied for n gears shifted so that cumulative errors caused by dealing with integer rotation steps are corrected.
- fixed motor fault EXTI handling
- added arrays for Iprop and IpropRate; modified ISR to collect & compute those values
- added the possibility to measure magnetic gear rotation either by counting as5601's A channel EXITs or by reading its raw angle register via I2C
implemented this change in mj514.c, gear.c

in mj514_adc.c:
- added typecasts to avoid compiler warnings

in gear.c:
- added a while() loop to have some from of atomic shifting

in mj514.c/.h:
- increased timer16 ISR priority by 1
- sorted out the interrupt priority mess

in mb85rc.c:
- modified code so that this driver can work with 2-byte wide FeRAM register addresses
- changed type of RegAddr from uint8_t to uint16_t (as it should be)

in button.c & composite_led_actual.c:
- added #if defined(USE_BUTTON) and USE_LED

in event.c:
- replaced e.g. #if (MJ808_) with #if defined(MJ808_)
- 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
Parts:
- removed R902: foo, rcl:R0402
- added C805: 0.22uF / 50V, rcl:C0402
- added R803: 10k, rcl:R0402
- R801: device rcl:R0603 -> rcl:R0402
- moved R801 0.25 mm to (4.00, 6.75)
Connections:
- removed net MC:PMODE: IC901.P$14, R902.2
- removed net STM32F04:PA5: IC302.11_PA5
- new net 12V0:!SHDN!_IN: C805.1, IC801.!SHDN!, R803.1
- new net 12V0_!SHDN!: IC302.11_PA5, R803.2
- net 3V3: now also IC901.P$14
- net BAT+: no longer IC801.!SHDN!
- net GND: now also C805.2; no longer R902.1
Routing:
- net 12V0:!SHDN!_IN: track 0.00 -> 43.2 mm, vias 0 -> 2
- net GND: track 9.04 -> 13.9 mm, vias 40 -> 39
- net 12V0_!SHDN!: track 0.00 -> 2.73 mm
- net 3V3: track 31.6 -> 34.3 mm, vias 15 -> 16
- net MC:PMODE: track 1.29 -> 0.00 mm
- net MOTOR_IN1: track 20.3 -> 21.3 mm
Other:
- board text added: "MJ514 ejovrh rev.1a"
- board text removed: "MJ514 ejovrh rev.1"
