File: eagle design/mj514/MJ514 - rev.1 - prod.sch (EAGLE design)
At the start: 4 parts

Commit message: MJ818 SuperNova Mini2: - added position key into PCB and spacers; updated gerber, dwg and stl
mj513 - grip:
- corrected bushing dimensions

in mj8x8-foo:
- minor corrections

general board-wide effort:
- replaced pinhead with 0.9mm TH
- added 2nd CAN H & L solder contact
- unified sch nets and drawings

in mj8x8 foo:
- developed rev.1b mj-foo device with voltage detector and CAN TVS protection

in mj808 design:
- updated front led shunt resistor to 0.18 Ohm

in mj8x8:
- added HR30-6R-6P - PushPull Receptacle.lbr receptable
Parts:
- removed JP1, JP2, JP3: (no value), pinhead:PINHD-1X2
- added CONN1: HR30-6R-6P(71), HR30-6R-6P - PushPull Receptacle:HR-30-6R-6X
- added TP1: LiIon + Terminal, signal testpoint:TPTH-0.9
- added TP2: LiIon - Terminal, signal testpoint:TPTH-0.9
- added TP3: motor +, signal testpoint:TPTH-0.9
- added TP4: motor -, signal testpoint:TPTH-0.9
- added TP5, TP7: CAN high, signal testpoint:TPTH-0.9
- added TP6, TP8: CAN low, signal testpoint:TPTH-0.9
Connections:
- net BAT+: now also CONN1.6, TP1.TP$1; no longer JP2.2
- net CAN_H: now also CONN1.4, CONN1.5, TP5.TP$1, TP7.TP$1; no longer JP3.1
- net CAN_L: now also CONN1.2, CONN1.3, TP6.TP$1, TP8.TP$1; no longer JP3.2
- net GND: now also CONN1.1, TP2.TP$1; no longer JP2.1
- net MOTOR+: now also TP3.TP$1; no longer JP1.1
- net MOTOR-: now also TP4.TP$1; no longer JP1.2
Other:
- note added: "2"
- note added: "3"
- note added: "4"
- note added: "Rohloff E14 servo controller HW rev.1"
- note added: "inbound, brown"
- note added: "inbound, white"
- note added: "outbound, brown"
- note added: "outbound, white"

Commit message: mj514 prod work: - essentially copied POC sch & brd - added SHT40-AD1F - Humidity Sensor to POC and prod boards - converted to 6 layer board - ERC & DRC check out ok - created gerbers
Parts:
- added R1, R2: 4k7, rcl:R-EU_R0402
- TP3: value motor + -> CAN high
- TP4: value motor - -> CAN high
- TP5: value CAN high -> CAN low
- TP7: value CAN high -> motor +
- TP8: value CAN low -> motor -
Connections:
- new net 12V: R2.2
- new net EN: R1.2
- new net FB: R1.2, R2.1
- new net I2C_SCL: R1.1
- new net I2C_SDA: R2.1
- new net IMODE: R1.2
- new net L: R2.1
- new net PMODE: R2.2
- new net SPLIT: R2.2
- net 3V3: now also R1.2, R2.2
- net BAT+: now also R1.1
- net CAN_H: now also TP3.TP$1, TP4.TP$1; no longer TP5.TP$1, TP7.TP$1
- net CAN_L: now also TP5.TP$1; no longer TP8.TP$1
- net GND: now also R1.1, R2.1
- net MOTOR+: now also TP7.TP$1; no longer TP3.TP$1
- net MOTOR-: now also TP8.TP$1; no longer TP4.TP$1
Other:
- note added: "5"
- note added: "6"
- note added: "7"
- note added: "9"
- note added: "FB Resistors: VOUT = 1.265V(1 + R1/R2). 12V = 1.265V * (1 + 85.8/10) = 12.09V"
- note added: "Inductor: DS. p. 5: L = 3 (VIN/VOUT) (VOUT – VIN)/(IMAX • f) 8.4V: L= 3 * (8.4/12.0) * (12.0 - 8.4) / (1.5A * 1.2MHz) = 3 * 0.7 / (1.5 * 1.2exp6) = 3 * 3.89exp-7 = 1.17 uH 7.0V: L= 3 * (7/12.0) * (12.0 - 7.0) / (1.5A * 1.2MHz) = 3 * 0.5833 / (1.5 * 1.2exp6) = 3 * 3.24exp-7 = 9.72 uH"
- note added: "Vmotor_iprop (ADC input): V = R * I = 1k * 1A = 1V"
- note added: "low-pass fcutoff 723.4 Hz"
- note added: "see DS. p. 13"
- moved on the sheet: TP1, TP2, TP3, TP4, TP5, TP6, TP7, TP8

Commit message: in board design: - added current sense resistor calculation - in 12V0 regulator added slow start RC lowpass filter, as per DS. p. 6 - moved 12V_SHDN to PA5
in motor.c/.h:
- code tweaks for angle statistics
- added #if USE_AS5601_PULSE across the code to deactivate not needed code
- in timer16 ISR: added _EndTravelTime and coded setting this variable with the elapsed milliseconds once the travel end is reached
- in timer16 ISR: added code which allows timer16 to continue to run after end travel is reached
- in _StartMotorController() & _StopMotorController() added timer16 interrupt priority change (suspect was some race condition or priority collision)
- set & unset FlagShiftingDone, for above checks
- added #define USE_RAMPUP so that rampup code can be disabled
- cleaned up code by adding #if CURRENT_STATS and #if ANGLE_STATS
- added typecast to get rid of compiler warnings
- added misc. code for testing stuff
- added arrays _PulseCorrection[] and _RawAngleCorrection; these hold corrections which need to be applied for n gears shifted so that cumulative errors caused by dealing with integer rotation steps are corrected.
- fixed motor fault EXTI handling
- added arrays for Iprop and IpropRate; modified ISR to collect & compute those values
- added the possibility to measure magnetic gear rotation either by counting as5601's A channel EXITs or by reading its raw angle register via I2C
implemented this change in mj514.c, gear.c

in mj514_adc.c:
- added typecasts to avoid compiler warnings

in gear.c:
- added a while() loop to have some from of atomic shifting

in mj514.c/.h:
- increased timer16 ISR priority by 1
- sorted out the interrupt priority mess

in mb85rc.c:
- modified code so that this driver can work with 2-byte wide FeRAM register addresses
- changed type of RegAddr from uint8_t to uint16_t (as it should be)

in button.c & composite_led_actual.c:
- added #if defined(USE_BUTTON) and USE_LED

in event.c:
- replaced e.g. #if (MJ808_) with #if defined(MJ808_)
- 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
Connections:
- removed net PMODE: R2.2
- net GND: no longer R2.1
Other:
- note added: "8"
- note added: "Pmode = HIGH -- DS. p. 11 controller is in PWM Control Mode"
- note added: "Rohloff E14 servo controller HW rev.1a"
- note added: "Vmotor_iprop (ADC input) resistor: DS. p. 12 & 13 Vref is 3.3V R=1k: 3.3A R=1k886: 1.75A R=2k: 1.65A R=2k2: 1.5A"
- note added: "soft start: DS. p. 6 fcutoff = 72.3Hz"
- note removed: "Rohloff E14 servo controller HW rev.1"
- note removed: "Vmotor_iprop (ADC input): V = R * I = 1k * 1A = 1V"
