File: eagle design/mj514/MJ514 - rev.1a - prod.sch (EAGLE design)
At the start: 12 parts

Commit message: ///////// start of HW Rev.1a ///////// !!! board design is not true hw rev.1a - was manually edited to match actual oshpark fabrication!!!
in mj838.c/.h:
- adapted base hw rev.1 code to hw rev.1a board: moved CAN standby GPIO to PA15

in motor.c/.h:
- manual merge of "raw angles per ms" branch

in board design:
- removed not prod related designs & schematics
- added motor controller Pmode resistor so that oshpark delivered board matches with drawing ( minus 12V0 regulator shutdown line - this still exists in this board)
- moved AS5601 0.5mm east and corrected 3V3 via position
- corrected tplace via markings
- corrected dimensions: N +=0.5mm, E += 1mm
- corrected E screw via hole += 1mm towards N and += 2mm towards E
- rounded a few corners
- in motor controller sheet changed value of Iprop resistor from 1k to 2k2
- added debug0/1/2 GPIOs on PB0/1 & PA7
- moved semi-circular cutout at NE side of board 1mm towards E
- added vias for SWD & 2V2/GND wired connections to programming adapter

board sent to fab
Parts:
- added 3V3, DEBUG0, DEBUG1, DEBUG2, GND, MOTOR_FLT, MOTOR_IPROP, SWCLK, SWDIO: TP0.6, TP-06:TP0.6
- CONN1: value HR30-6R-6P(71) -> HR30-6JA-6P71
Connections:
- new net DEBUG0: DEBUG0.P$1
- new net DEBUG1: DEBUG1.P$1
- new net DEBUG2: DEBUG2.P$1
- new net MOTOR_FLT: MOTOR_FLT.P$1
- new net MOTOR_IPROP: MOTOR_IPROP.P$1
- new net PMODE: R2.2
- net 3V3: now also 3V3.P$1
- net GND: now also GND.P$1, R2.1
- net SYS_SWCLK: now also SWCLK.P$1
- net SYS_SWDIO: now also SWDIO.P$1
Other:
- note added: "jack, mounted on existing Rohloff e514 6-lead cable"
