File: eagle design/mj000/Nucleo-F042K6 - mj8x8 gateway- rev.1 - TCAN334 - poc.brd (EAGLE design)
At the start: 20 x 40 mm, 16 parts, among them IC201 ADXL367, IC301 47309-2651, IC401 TCAN334, J1 Batt, J2 Batt

Commit message: some forgotten work from half a year ago
Connections:
- removed net PA10: JP1.2
- new net PA2: JP2.5
- net ADXL367_CS: now also JP1.2; no longer JP2.5
Routing:
- net 3V3: track 55.7 -> 50.7 mm
- net ADXL367_CS: track 10.8 -> 11.7 mm, vias 0 -> 1
Changed lines of the file:
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@@
 <via x="-1.25" y="33" extent="1-16" drill="0.35"/>
 <via x="1.25" y="38.5" extent="1-16" drill="0.35"/>
-<wire x1="1.25" y1="33" x2="1.25" y2="38.5" width="0.25" layer="16"/>
+<wire x1="2" y1="37.75" x2="1.25" y2="38.5" width="0.25" layer="16"/>
+<wire x1="2" y1="37.75" x2="2" y2="33" width="0.25" layer="16"/>
 <wire x1="-0.9" y1="34.5" x2="-0.9" y2="34.1" width="0.25" layer="1"/>
 <wire x1="-0.9" y1="34.1" x2="-1.25" y2="33.75" width="0.25" layer="1"/>
@@
 <wire x1="1.25" y1="38.25" x2="1.25" y2="38.5" width="0.25" layer="1"/>
 <wire x1="-1.25" y1="33" x2="0" y2="33" width="0.25" layer="16"/>
-<wire x1="0" y1="33" x2="1.25" y2="33" width="0.25" layer="16"/>
-<wire x1="3.25" y1="28.75" x2="2" y2="28.75" width="0.25" layer="16"/>
-<wire x1="2" y1="28.75" x2="1.25" y2="29.5" width="0.25" layer="16"/>
-<wire x1="1.25" y1="38.5" x2="1.25" y2="29.5" width="0.25" layer="16"/>
+<wire x1="0" y1="33" x2="2" y2="33" width="0.25" layer="16"/>
+<wire x1="3.25" y1="28.75" x2="2.5" y2="28.75" width="0.25" layer="16"/>
 <wire x1="0" y1="32.9" x2="0" y2="33" width="0.25" layer="1"/>
+<wire x1="2" y1="33" x2="2" y2="29.25" width="0.25" layer="16"/>
+<wire x1="2" y1="29.25" x2="2.5" y2="28.75" width="0.25" layer="16"/>
 </signal>
 <signal name="TXCAN" class="3">
@@
 <signal name="PA9">
 <contactref element="JP1" pad="1"/>
-</signal>
-<signal name="PA10">
-<contactref element="JP1" pad="2"/>
 </signal>
 <signal name="PB0">
@@
 <contactref element="JP1" pad="3"/>
 <wire x1="-7.62" y1="37.846" x2="7.62" y2="37.846" width="0" layer="19" extent="1-1"/>
-</signal>
-<signal name="PA8" class="3">
-<contactref element="JP1" pad="12"/>
 </signal>
 <signal name="CAN_INFRA:SPLIT" class="3">
@@
 <contactref element="R202" pad="1"/>
 <wire x1="0.9" y1="36" x2="0.9" y2="36.4" width="0.25" layer="1"/>
-<wire x1="1.25" y1="36.75" x2="1.25" y2="37.25" width="0.25" layer="1"/>
+<wire x1="1.25" y1="36.75" x2="1.25" y2="37" width="0.25" layer="1"/>
 <wire x1="1.25" y1="36.75" x2="0.9" y2="36.4" width="0.25" layer="1"/>
-<contactref element="JP2" pad="5"/>
-<wire x1="0.9" y1="36" x2="4.75" y2="36" width="0.25" layer="1"/>
-<wire x1="5.25" y1="33.25" x2="5.75" y2="32.75" width="0.25" layer="1"/>
-<wire x1="5.75" y1="32.75" x2="7.604" y2="32.75" width="0.25" layer="1"/>
-<wire x1="7.604" y1="32.75" x2="7.62" y2="32.766" width="0.25" layer="1"/>
-<wire x1="4.75" y1="36" x2="5.25" y2="35.5" width="0.25" layer="1"/>
-<wire x1="5.25" y1="35.5" x2="5.25" y2="33.25" width="0.25" layer="1"/>
+<contactref element="JP1" pad="2"/>
+<via x="1.25" y="37" extent="1-16" drill="0.35"/>
+<wire x1="-7.62" y1="40.386" x2="-3.136" y2="40.386" width="0.25" layer="16"/>
+<wire x1="0.25" y1="37" x2="1.25" y2="37" width="0.25" layer="16"/>
+<wire x1="-3.136" y1="40.386" x2="0.25" y2="37" width="0.25" layer="16"/>
+<wire x1="1.25" y1="37.25" x2="1.25" y2="37" width="0.25" layer="1"/>
 </signal>
 <signal name="SD_CS">
@@
 <contactref element="IC201" pad="9"/>
 </signal>
+<signal name="PA2">
+<contactref element="JP2" pad="5"/>
+</signal>
+<signal name="PA8">
+<contactref element="JP1" pad="12"/>
+</signal>
 </signals>
