File: eagle design/mj000/Nucleo-F042K6 - mj8x8 gateway- rev.1 - TCAN334 - poc.sch (EAGLE design)
At the start: 4 parts, among them J1 Batt, J2 Batt

Commit message: some forgotten work from half a year ago
Connections:
- removed net PA10: JP1.2
- new net PA2: JP2.5
- net ADXL367_CS: now also JP1.2; no longer JP2.5
Changed lines of the file:
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@@
-</segment>
-</net>
-<net name="PA10" class="0">
-<segment>
-<pinref part="JP1" gate="A" pin="2"/>
-<wire x1="45.72" y1="139.7" x2="35.56" y2="139.7" width="0.1524" layer="91"/>
-<label x="35.56" y="139.7" size="1.778" layer="95" rot="R180"/>
 </segment>
 </net>
@@
 <wire x1="45.72" y1="137.16" x2="35.56" y2="137.16" width="0.1524" layer="91"/>
 <label x="35.56" y="137.16" size="1.778" layer="95" rot="R180"/>
-</segment>
-</net>
-<net name="PA8" class="3">
-<segment>
-<pinref part="JP1" gate="A" pin="12"/>
-<wire x1="45.72" y1="114.3" x2="35.56" y2="114.3" width="0.1524" layer="91"/>
-<label x="35.56" y="114.3" size="1.778" layer="95" rot="R180"/>
 </segment>
 </net>
@@
 </segment>
 <segment>
+<pinref part="JP1" gate="A" pin="2"/>
+<wire x1="45.72" y1="139.7" x2="35.56" y2="139.7" width="0.1524" layer="91"/>
+<label x="35.56" y="139.7" size="1.778" layer="95" rot="R180"/>
+</segment>
+</net>
+<net name="SD_CS" class="0">
+<segment>
+<portref moduleinst="SDCARD" port="SD_CS"/>
+<wire x1="180.34" y1="101.6" x2="162.56" y2="101.6" width="0.1524" layer="91"/>
+<label x="170.18" y="101.6" size="1.778" layer="95"/>
+</segment>
+<segment>
+<pinref part="JP2" gate="A" pin="10"/>
+<wire x1="76.2" y1="119.38" x2="86.36" y2="119.38" width="0.1524" layer="91"/>
+<label x="86.36" y="119.38" size="1.778" layer="95"/>
+</segment>
+</net>
+<net name="PA2" class="0">
+<segment>
 <pinref part="JP2" gate="A" pin="5"/>
 <wire x1="76.2" y1="132.08" x2="86.36" y2="132.08" width="0.1524" layer="91"/>
@@
 </segment>
 </net>
-<net name="SD_CS" class="0">
-<segment>
-<portref moduleinst="SDCARD" port="SD_CS"/>
-<wire x1="180.34" y1="101.6" x2="162.56" y2="101.6" width="0.1524" layer="91"/>
-<label x="170.18" y="101.6" size="1.778" layer="95"/>
-</segment>
-<segment>
-<pinref part="JP2" gate="A" pin="10"/>
-<wire x1="76.2" y1="119.38" x2="86.36" y2="119.38" width="0.1524" layer="91"/>
-<label x="86.36" y="119.38" size="1.778" layer="95"/>
-</segment>
-</net>
+<net name="PA8" class="0">
+<segment>
+<pinref part="JP1" gate="A" pin="12"/>
+<wire x1="45.72" y1="114.3" x2="35.56" y2="114.3" width="0.1524" layer="91"/>
+<label x="35.56" y="114.3" size="1.778" layer="95" rot="R180"/>
+</segment>
+</net>
