File: eagle design/mj838/GnZC/GnZC - POC.sch (EAGLE design)
At the start: 20 parts, among them IC1 MIC2514YM5

Commit message: in GnZC - POC.brd/sch: - changed 3V3 power symbol
Connections:
- net +3V3 renamed 3V3
