File: eagle design/mj8x8/MJ8x8 clone - rev.5 - TCAN334 - poc.sch (EAGLE design)
At the start: 3 parts, among them J1 CAN, J2 Power Supply

Commit message: - new programming adapter
Parts:
- removed SWD101: TC2030-NL, tag-connect:TC2030
- added J3: CAN, con-amp:MTA02-100
- J1: value CAN -> Power Supply
- J2: value Power Supply -> FTSH-107-01-L-DV-K-A; device con-amp:MTA02-100 -> STM32 JTAG 1.27mm 14pin header:FTSH-107-01-L-DV-K-A
Connections:
- net 3V3: now also J2.T_VCC_P3; no longer SWD101.1_T_VCC
- net BAT+: now also J1.2; no longer J2.2
- net CAN_H: now also J3.1; no longer J1.1
- net CAN_L: now also J3.2; no longer J1.2
- net GND: now also J1.1, J2.GND-DETECT_P11, J2.GND_P5, J2.GND_P7; no longer J2.1, SWD101.5_GND
- net SYS_NRST: now also J2.T_NRST_P12; no longer SWD101.3_T-NRST
- net SYS_SWCLK: now also J2.T_JCLK/T_SWCLK_P6; no longer SWD101.4_T-SWCLK
- net SYS_SWDIO: now also J2.TJTMS/T_SWDIO_P4; no longer SWD101.2_T-SWDIO
Other:
- note added: "MJ8??? - foo device"
- note removed: "MJ8???8 - foo device"
- moved on the sheet: J1

Commit message: MJ818 SuperNova Mini2: - added position key into PCB and spacers; updated gerber, dwg and stl
mj513 - grip:
- corrected bushing dimensions

in mj8x8-foo:
- minor corrections

general board-wide effort:
- replaced pinhead with 0.9mm TH
- added 2nd CAN H & L solder contact
- unified sch nets and drawings

in mj8x8 foo:
- developed rev.1b mj-foo device with voltage detector and CAN TVS protection

in mj808 design:
- updated front led shunt resistor to 0.18 Ohm

in mj8x8:
- added HR30-6R-6P - PushPull Receptacle.lbr receptable
Other:
- note added: "2"
- note added: "3"
- note added: "4"

Commit message: in all mj-devices: - seperated MJ8x8 clone - rev.5 - TCAN334 - poc.brd(generic) BOMs from device specific
Parts:
- removed J2: FTSH-107-01-L-DV-K-A, STM32 JTAG 1.27mm 14pin header:FTSH-107-01-L-DV-K-A
- removed J3: CAN, con-amp:MTA02-100
- added CONN1: HR30-6R-6P(71), HR30-6R-6P - PushPull Receptacle:HR-30-6R-6X
- added TP1: LiIon + Terminal, signal testpoint:TPTH-0.9
- added TP2: LiIon - Terminal, signal testpoint:TPTH-0.9
- added TP5, TP6: CAN high, signal testpoint:TPTH-0.9
- added TP7, TP8: CAN low, signal testpoint:TPTH-0.9
- J1: value Power Supply -> FTSH-107-01-L-DV-K-A; device con-amp:MTA02-100 -> STM32 JTAG 1.27mm 14pin header:FTSH-107-01-L-DV-K-A
Connections:
- net 3V3: now also J1.T_VCC_P3; no longer J2.T_VCC_P3
- net BAT+: now also CONN1.6, TP1.TP$1; no longer J1.2
- net CAN_H: now also CONN1.4, CONN1.5, TP5.TP$1, TP6.TP$1; no longer J3.1
- net CAN_L: now also CONN1.2, CONN1.3, TP7.TP$1, TP8.TP$1; no longer J3.2
- net GND: now also CONN1.1, J1.GND-DETECT_P11, J1.GND_P5, J1.GND_P7, TP2.TP$1; no longer J1.1, J2.GND-DETECT_P11, J2.GND_P5, J2.GND_P7
- net SYS_NRST: now also J1.T_NRST_P12; no longer J2.T_NRST_P12
- net SYS_SWCLK: now also J1.T_JCLK/T_SWCLK_P6; no longer J2.T_JCLK/T_SWCLK_P6
- net SYS_SWDIO: now also J1.TJTMS/T_SWDIO_P4; no longer J2.TJTMS/T_SWDIO_P4
Other:
- note added: "??? device HW rev.1"
- note added: "MJ???"
- note added: "MJ??? device"
- note added: "inbound, brown"
- note added: "inbound, white"
- note added: "outbound, brown"
- note added: "outbound, white"
- note removed: "MJ8??? - foo device"
