File: eagle design/mj838/MJ838 - rev.1b - TCAN334 - poc.sch (EAGLE design)
At the start: 27 parts, among them J1 Battery, J2 FTSH-107-01-L-DV-K-A, J3 CAN, J4 sense 1, J5 sense 2

Commit message: ////// start of MJ838 HW rev.1b //////
in spice simulation:
- in ZeroCross detection circuit, replaced OpAmp comparator with dedicated comparator, added OptoCoupler
- added experimental 2xNMos + OptoCoupler circuit for Zerocross detection

in brd & sch:
- added a bit of TVS/ESD protection for SWD, 3V3 bus
- in zerocross sheet, added 4N25 optocoupler to comparator output
- added INA219 - I2C Current & Power Monitor - as an alternative to the PAC1952
- replaced FeRAM module with different footprint, which in turn enables usage of modules of larger capacity
- resolved short between dynamo1 and 2: turns out, NC SSRs are not needed: replaced two NC SSRs with NO SSRs (SW1 and 2)
- corrected SSR control LED resistor
- replaced zero-cross LT1638 OpAmp with LT1716 comparator
- added RA connector: rev.1b layout with card edge connector & completely new board dimensions
- THE GREED! - converted to 6 layer PCB
- added non-inverting OpAmp for 10x Vsense amplification: 100mA load current gives 10mA Vsense. that amplified 10x gives 100mV Gate-Driver input, thus 100mV ADC output
- updated gerbers for rev.1b
- added more powerful PH2925U - N-Fet (lib and datasheet)
- added ltspice simulation adjustable load.asc
- added 20W 12R resistor (replaces too low-powered SMD version)
Parts:
- removed TP31: BAT+, signal testpoint:TPTH-0.9
- added TP1: TPPAD1-13, testpad:TPPAD1-13
Connections:
- removed net SMOOTHINGCAP_IN: R2.2
- removed net V_RECT_TP1-IN: R2.1
- new net N$1: R1.2
- net GND: now also R1.1
- net IN: no longer R1.2
- net LOAD_LOW: no longer R1.1
- net ZEROCROSS: now also TP1.TP; no longer TP31.TP$1
Other:
- note added: "Gate Driver"
- note added: "I2C control input"
- note added: "Load"
- note added: "Ohmic, constant"
- note added: "Rsense Volatge Drop U = R*I : 0.1 * 1A = 100mV 500mA load: 50mV 100mA load: 10mV 50mA load: 5mV and so on..."
- note added: "Vsense amplifier"
- note added: "Vsense range: 0 to approx. 100mV for a current of 0 to approx. 1A"
- note added: "mj838 - Čos - dynamo electrnics HW rev.1b"
- note added: "non-inverting, 1:10 ratio: Vout = Vin * (1+ 9k/1k) in (Vsense), out (Vsense-Amp_Out): 5mV -> 50mV 10mV -> 100mV 100mV -> 1V"
- note added: "not really ohmic, adjustable"
- note added: "required DAC output voltage: 0 to approx. 1V (matches the Vsense amplifier output range)"
- note added: "shunt, constant"
- note removed: "Rsense Volatge Drop U = R*I : 0.1 * 1A = 100mV 500mA load: 50mV 100mA load: 10mV and so on..."
- note removed: "TP1"
- note removed: "TP2"
- note removed: "Vsense range: 0 to approx. 100mV"
- note removed: "e.g. CPA2512Q12R0FS-T10"
- note removed: "e.g. WSL2512R1000DEA"
- note removed: "for direct N-Fet <-> GPIO control use IRLML2402TRPBF for OpAmp/DAC control use SI2316BDS-T1-E3"
- note removed: "mj838 - Čos - dynamo electrnics HW rev.1a"
- note removed: "required DAC output voltage: 0 to approx. 100mV"

Commit message: HW rev.1a finished
in mj838.brd/.sch:
- added adjustable current sink by means of a N-Fet gate driven by an opamp, in turn controlled by a voltage supplied by a a I2C controlled DAC connected to the opamp's inverting input.
- moved almost all elements to top layer. exceptions are for now SSRs.
- added DAC121C081 - 12bit I2C DAC datasheet and eagle lib
- added TName indicators for easier probing of SSD relay contact points between TLC59208F and SSR LED cathode
- reconfigured 12R artifical load to permanently have a 12R SMD resistor on board
- added application load which has a screw terminal and N-Fet power control
- updated BOM MJ838 - rev.1 - TCAN334 - poc.xlsx
- replaced pac1952-1 with correct pac1952-2
- added ZC testpin
- added labels to I2C nets in stm32 sheet
- replaced high-side load switch with n-fet
- replaced Battery/ground TH testpad with terminal block connector
- added CAN terminal block connector in parallel to TH testpads
- replaced PAC1954 TH testpads with terminal block connectors

in PAC1954 - Power Monitor.lbr:
- corrected the whole lib in respect to PAC195x-1/-2 differences
Parts:
- removed TP1: TPPAD1-13, testpad:TPPAD1-13
- added TP31: BAT+, signal testpoint:TPTH-0.9
Connections:
- removed net N$1: R1.2
- new net SMOOTHINGCAP_IN: R2.2
- new net V_RECT_TP1-IN: R2.1
- net GND: no longer R1.1
- net IN: now also R1.2
- net LOAD_LOW: now also R1.1
- net ZEROCROSS: now also TP31.TP$1; no longer TP1.TP
Other:
- note added: "Rsense Volatge Drop U = R*I : 0.1 * 1A = 100mV 500mA load: 50mV 100mA load: 10mV and so on..."
- note added: "TP1"
- note added: "TP2"
- note added: "Vsense range: 0 to approx. 100mV"
- note added: "e.g. CPA2512Q12R0FS-T10"
- note added: "e.g. WSL2512R1000DEA"
- note added: "for direct N-Fet <-> GPIO control use IRLML2402TRPBF for OpAmp/DAC control use SI2316BDS-T1-E3"
- note added: "mj838 - Čos - dynamo electrnics HW rev.1a"
- note added: "required DAC output voltage: 0 to approx. 100mV"
- note removed: "Gate Driver"
- note removed: "I2C control input"
- note removed: "Load"
- note removed: "Ohmic, constant"
- note removed: "Rsense Volatge Drop U = R*I : 0.1 * 1A = 100mV 500mA load: 50mV 100mA load: 10mV 50mA load: 5mV and so on..."
- note removed: "Vsense amplifier"
- note removed: "Vsense range: 0 to approx. 100mV for a current of 0 to approx. 1A"
- note removed: "mj838 - Čos - dynamo electrnics HW rev.1b"
- note removed: "non-inverting, 1:10 ratio: Vout = Vin * (1+ 9k/1k) in (Vsense), out (Vsense-Amp_Out): 5mV -> 50mV 10mV -> 100mV 100mV -> 1V"
- note removed: "not really ohmic, adjustable"
- note removed: "required DAC output voltage: 0 to approx. 1V (matches the Vsense amplifier output range)"
- note removed: "shunt, constant"
